File: pcb/Amplifier.kicad_sch (KiCad schematic)
At the start: 23 parts, among them J4 Screw_Terminal_01x04, U9 MA12040PXUMA1

Commit message: - work in progress, changed rj45 connector
Parts:
- renumbered U9 to U8
Changed lines of the file:
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@@
         )
         (path "/c639bae0-d26f-43ee-9e8c-ca060284bd0b/ecbd0217-ab04-4196-9487-2acaa32ad17c"
-          (reference "#PWR034") (unit 1)
+          (reference "#PWR035") (unit 1)
         )
       )
@@
         )
         (path "/c639bae0-d26f-43ee-9e8c-ca060284bd0b/ecbd0217-ab04-4196-9487-2acaa32ad17c"
-          (reference "#PWR029") (unit 1)
+          (reference "#PWR030") (unit 1)
         )
       )
@@
         )
         (path "/c639bae0-d26f-43ee-9e8c-ca060284bd0b/ecbd0217-ab04-4196-9487-2acaa32ad17c"
-          (reference "TP17") (unit 1)
+          (reference "TP19") (unit 1)
         )
       )
@@
         )
         (path "/c639bae0-d26f-43ee-9e8c-ca060284bd0b/ecbd0217-ab04-4196-9487-2acaa32ad17c"
-          (reference "TP16") (unit 1)
+          (reference "TP18") (unit 1)
         )
       )
@@
         )
         (path "/c639bae0-d26f-43ee-9e8c-ca060284bd0b/ecbd0217-ab04-4196-9487-2acaa32ad17c"
-          (reference "#PWR036") (unit 1)
+          (reference "#PWR037") (unit 1)
         )
       )
@@
         )
         (path "/c639bae0-d26f-43ee-9e8c-ca060284bd0b/ecbd0217-ab04-4196-9487-2acaa32ad17c"
-          (reference "TP14") (unit 1)
+          (reference "TP16") (unit 1)
         )
       )
@@
   (symbol (lib_id "MA12040PXUMA1:MA12040PXUMA1") (at 125.73 96.52 0) (unit 1)
     (in_bom yes) (on_board yes) (dnp no) (fields_autoplaced)
-    (property "Reference" "U9" (at 125.73 45.72 0)
+    (property "Reference" "U8" (at 125.73 45.72 0)
       (effects (font (size 1.27 1.27)))
     )
@@
       (project "VolumioAmp"
         (path "/c639bae0-d26f-43ee-9e8c-ca060284bd0b/ecbd0217-ab04-4196-9487-2acaa32ad17c"
-          (reference "U9") (unit 1)
+          (reference "U8") (unit 1)
         )
       )
@@
         )
         (path "/c639bae0-d26f-43ee-9e8c-ca060284bd0b/ecbd0217-ab04-4196-9487-2acaa32ad17c"
-          (reference "#PWR031") (unit 1)
+          (reference "#PWR032") (unit 1)
         )
       )
@@
         )
         (path "/c639bae0-d26f-43ee-9e8c-ca060284bd0b/ecbd0217-ab04-4196-9487-2acaa32ad17c"
-          (reference "#PWR030") (unit 1)
+          (reference "#PWR031") (unit 1)
         )
       )
@@
         )
         (path "/c639bae0-d26f-43ee-9e8c-ca060284bd0b/ecbd0217-ab04-4196-9487-2acaa32ad17c"
-          (reference "#PWR035") (unit 1)
+          (reference "#PWR036") (unit 1)
         )
       )
@@
         )
         (path "/c639bae0-d26f-43ee-9e8c-ca060284bd0b/ecbd0217-ab04-4196-9487-2acaa32ad17c"
-          (reference "#PWR033") (unit 1)
+          (reference "#PWR034") (unit 1)
         )
       )
@@
         )
         (path "/c639bae0-d26f-43ee-9e8c-ca060284bd0b/ecbd0217-ab04-4196-9487-2acaa32ad17c"
-          (reference "#PWR032") (unit 1)
+          (reference "#PWR033") (unit 1)
         )
       )
@@
         )
         (path "/c639bae0-d26f-43ee-9e8c-ca060284bd0b/ecbd0217-ab04-4196-9487-2acaa32ad17c"
-          (reference "TP13") (unit 1)
+          (reference "TP15") (unit 1)
         )
       )
@@
         )
         (path "/c639bae0-d26f-43ee-9e8c-ca060284bd0b/ecbd0217-ab04-4196-9487-2acaa32ad17c"
-          (reference "TP18") (unit 1)
+          (reference "TP20") (unit 1)
         )
       )
@@
         )
         (path "/c639bae0-d26f-43ee-9e8c-ca060284bd0b/ecbd0217-ab04-4196-9487-2acaa32ad17c"
-          (reference "TP15") (unit 1)
-        )
-      )
+          (reference "TP17") (unit 1)
+        )
+      )
