File: pcb/Amplifier.kicad_sch (KiCad schematic)
At the start: 23 parts, among them J4 Screw_Terminal_01x04, U8 MA12040PXUMA1

Commit message: - component placed
Parts:
- added L2, L3, L4, L5: L, symbol Device:L
Connections:
- net +5v: now also U8.17 (AVDD)
- net GND: no longer U8.17 (AVDD)
- net at U8.4 (OUT0A), U8.5 (OUT0A): now also J4.2 (Pin_2); no longer J4.1 (Pin_1)
- net at U8.10 (OUT0B), U8.11 (OUT0B): now also J4.1 (Pin_1); no longer J4.2 (Pin_2)
- net at U8.44 (OUT1A), U8.45 (OUT1A): now also J4.4 (Pin_4); no longer J4.3 (Pin_3)
- net at U8.38 (OUT1B), U8.39 (OUT1B): now also J4.3 (Pin_3); no longer J4.4 (Pin_4)
Other:
- moved on the sheet: C27

Commit message: - routed
Parts:
- added C27 (x4): 1u, Capacitor_SMD:C_0805_2012Metric_Pad1.18x1.45mm_HandSolder, symbol Device:C
- L2, L3, L4, L5: footprint (none) -> Inductor_SMD:L_0805_2012Metric
- TP5: footprint TestPoint:TestPoint_Bridge_Pitch2.54mm_Drill1.0mm -> TestPoint:TestPoint_Bridge_Pitch2.0mm_Drill0.7mm
Connections:
- net GND: now also C27.1, C27.1, C27.1, C27.1
- net at L4.1: now also U8.44 (OUT1A), U8.45 (OUT1A)
- net at L4.2: now also J4.4 (Pin_4), C27.2
- net at L5.1: now also U8.38 (OUT1B), U8.39 (OUT1B)
- net at L5.2: now also J4.3 (Pin_3), C27.2
- net at U8.10 (OUT0B), U8.11 (OUT0B): now also L3.1; no longer J4.1 (Pin_1)
- net at U8.4 (OUT0A), U8.5 (OUT0A): now also L2.1; no longer J4.2 (Pin_2)
- net at L3.2: now also J4.1 (Pin_1), C27.2
- net at L2.2: now also J4.2 (Pin_2), C27.2
Other:
- moved on the sheet: L2, L3, L4, L5

Commit message: - routed
Changed lines of the file:
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@@
     (stroke (width 0) (type default))
   )
-  (label "AC.~{ENABLE}" (at 105.41 124.46 0) (fields_autoplaced)
+  (label "AC.~{ENABLE}" (at 95.25 124.46 0) (fields_autoplaced)
     (effects (font (size 1.27 1.27)) (justify left bottom))
   )
-  (label "AC.~{MUTE}" (at 105.41 121.92 0) (fields_autoplaced)
+  (label "AC.~{MUTE}" (at 95.25 121.92 0) (fields_autoplaced)
     (effects (font (size 1.27 1.27)) (justify left bottom))
   )
@@
     (effects (font (size 1.27 1.27)) (justify left bottom))
   )
-  (label "AC.~{CLIP}" (at 105.41 127 0) (fields_autoplaced)
+  (label "AC.~{CLIP}" (at 95.25 127 0) (fields_autoplaced)
     (effects (font (size 1.27 1.27)) (justify left bottom))
   )
@@
     (effects (font (size 1.27 1.27)) (justify left bottom))
   )
-  (label "AC.~{ERROR}" (at 105.41 129.54 0) (fields_autoplaced)
+  (label "AC.~{ERROR}" (at 95.25 129.54 0) (fields_autoplaced)
     (effects (font (size 1.27 1.27)) (justify left bottom))
   )

Commit message: - BOM added (Farnell nrs)
Parts:
- C27: Farnell (none) -> 3013482
- C27: Farnell (none) -> 2611943
- C27: Farnell (none) -> 1414664
- C30: Farnell (none) -> 4146798
- J4: Farnell (none) -> 4179100
- L2, L3, L4, L5: value L -> 0.5u; footprint Inductor_SMD:L_0805_2012Metric -> Inductor_SMD:L_Bourns_SRN6045TA; Farnell (none) -> 3780754
- U8: Farnell (none) -> 2947805
Changed lines of the file:
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@@
+      (effects (font (size 1.27 1.27)) hide)
+    )
+    (property "Farnell" "3013482" (at 95.25 73.66 0)
       (effects (font (size 1.27 1.27)) hide)
     )
@@
       (effects (font (size 1.27 1.27)))
     )
-    (property "Value" "L" (at 166.37 106.68 90)
-      (effects (font (size 1.27 1.27)))
-    )
-    (property "Footprint" "Inductor_SMD:L_0805_2012Metric" (at 166.37 109.22 0)
+    (property "Value" "0.5u" (at 166.37 106.68 90)
+      (effects (font (size 1.27 1.27)))
+    )
+    (property "Footprint" "Inductor_SMD:L_Bourns_SRN6045TA" (at 166.37 109.22 0)
       (effects (font (size 1.27 1.27)) hide)
     )
     (property "Datasheet" "~" (at 166.37 109.22 0)
+      (effects (font (size 1.27 1.27)) hide)
+    )
+    (property "Farnell" "3780754" (at 166.37 109.22 0)
       (effects (font (size 1.27 1.27)) hide)
     )
@@
       (effects (font (size 1.27 1.27)) hide)
     )
+    (property "Farnell" "2611943" (at 156.21 111.76 0)
+      (effects (font (size 1.27 1.27)) hide)
+    )
     (pin "1")
     (pin "2")
@@
       (effects (font (size 1.27 1.27)))
     )
-    (property "Value" "L" (at 166.37 116.84 90)
-      (effects (font (size 1.27 1.27)))
-    )
-    (property "Footprint" "Inductor_SMD:L_0805_2012Metric" (at 166.37 119.38 0)
+    (property "Value" "0.5u" (at 166.37 116.84 90)
+      (effects (font (size 1.27 1.27)))
+    )
+    (property "Footprint" "Inductor_SMD:L_Bourns_SRN6045TA" (at 166.37 119.38 0)
       (effects (font (size 1.27 1.27)) hide)
     )
@@
       (effects (font (size 1.27 1.27)) hide)
     )
+    (property "Farnell" "3780754" (at 166.37 119.38 0)
+      (effects (font (size 1.27 1.27)) hide)
+    )
     (pin "1")
     (pin "2")
@@
     )
     (property "Datasheet" "~" (at 171.45 92.71 0)
+      (effects (font (size 1.27 1.27)) hide)
+    )
+    (property "Farnell" "3013482" (at 171.45 92.71 0)
       (effects (font (size 1.27 1.27)) hide)
     )
@@
     )
     (property "Datasheet" "~" (at 161.29 76.2 0)
+      (effects (font (size 1.27 1.27)) hide)
+    )
+    (property "Farnell" "3013482" (at 161.29 76.2 0)
       (effects (font (size 1.27 1.27)) hide)
     )
@@
       (effects (font (size 1.27 1.27)) hide)
     )
+    (property "Farnell" "4146798" (at 219.71 58.42 0)
+      (effects (font (size 1.27 1.27)) hide)
+    )
     (pin "1")
     (pin "2")
@@
       (effects (font (size 1.27 1.27)) hide)
     )
+    (property "Farnell" "2611943" (at 156.21 101.6 0)
+      (effects (font (size 1.27 1.27)) hide)
+    )
     (pin "1")
     (pin "2")
@@
     )
     (property "Datasheet" "~" (at 171.45 113.03 0)
+      (effects (font (size 1.27 1.27)) hide)
+    )
+    (property "Farnell" "3013482" (at 171.45 113.03 0)
       (effects (font (size 1.27 1.27)) hide)
     )
@@
       (effects (font (size 1.27 1.27)) hide)
     )
+    (property "Farnell" "4179100" (at 191.77 104.14 0)
+      (effects (font (size 1.27 1.27)) hide)
+    )
     (pin "3")
     (pin "2")
@@
       (effects (font (size 1.27 1.27)) hide)
     )
+    (property "Farnell" "2611943" (at 156.21 121.92 0)
+      (effects (font (size 1.27 1.27)) hide)
+    )
     (pin "1")
     (pin "2")
@@
       (effects (font (size 1.27 1.27)) hide)
     )
+    (property "Farnell" "3013482" (at 171.45 102.87 0)
+      (effects (font (size 1.27 1.27)) hide)
+    )
     (pin "1")
     (pin "2")
@@
       (effects (font (size 1.27 1.27)) hide)
     )
+    (property "Farnell" "3013482" (at 153.67 73.66 0)
+      (effects (font (size 1.27 1.27)) hide)
+    )
     (pin "1")
     (pin "2")
@@
     )
     (property "Datasheet" "~" (at 212.09 58.42 0)
+      (effects (font (size 1.27 1.27)) hide)
+    )
+    (property "Farnell" "3013482" (at 212.09 58.42 0)
       (effects (font (size 1.27 1.27)) hide)
     )
@@
       (effects (font (size 1.27 1.27)) hide)
     )
+    (property "Farnell" "3013482" (at 171.45 123.19 0)
+      (effects (font (size 1.27 1.27)) hide)
+    )
     (pin "1")
     (pin "2")
@@
     (property "MANUFACTURER" "Infineon Technologies" (at 125.73 96.52 0)
       (effects (font (size 1.27 1.27)) (justify bottom) hide)
+    )
+    (property "Farnell" "2947805" (at 125.73 96.52 0)
+      (effects (font (size 1.27 1.27)) hide)
     )
     (pin "38")
@@
       (effects (font (size 1.27 1.27)) hide)
     )
+    (property "Farnell" "2611943" (at 156.21 91.44 0)
+      (effects (font (size 1.27 1.27)) hide)
+    )
     (pin "1")
     (pin "2")
@@
       (effects (font (size 1.27 1.27)) hide)
     )
+    (property "Farnell" "3013482" (at 153.67 60.96 0)
+      (effects (font (size 1.27 1.27)) hide)
+    )
     (pin "1")
     (pin "2")
@@
     )
     (property "Datasheet" "~" (at 95.25 68.58 0)
+      (effects (font (size 1.27 1.27)) hide)
+    )
+    (property "Farnell" "3013482" (at 95.25 68.58 0)
       (effects (font (size 1.27 1.27)) hide)
     )
@@
       (effects (font (size 1.27 1.27)) hide)
     )
+    (property "Farnell" "1414664" (at 95.25 83.82 0)
+      (effects (font (size 1.27 1.27)) hide)
+    )
     (pin "1")
     (pin "2")
@@
       (effects (font (size 1.27 1.27)))
     )
-    (property "Value" "L" (at 166.37 96.52 90)
-      (effects (font (size 1.27 1.27)))
-    )
-    (property "Footprint" "Inductor_SMD:L_0805_2012Metric" (at 166.37 99.06 0)
+    (property "Value" "0.5u" (at 166.37 96.52 90)
+      (effects (font (size 1.27 1.27)))
+    )
+    (property "Footprint" "Inductor_SMD:L_Bourns_SRN6045TA" (at 166.37 99.06 0)
       (effects (font (size 1.27 1.27)) hide)
     )
@@
       (effects (font (size 1.27 1.27)) hide)
     )
+    (property "Farnell" "3780754" (at 166.37 99.06 0)
+      (effects (font (size 1.27 1.27)) hide)
+    )
     (pin "1")
     (pin "2")
@@
       (effects (font (size 1.27 1.27)) hide)
     )
+    (property "Farnell" "3013482" (at 162.56 63.5 0)
+      (effects (font (size 1.27 1.27)) hide)
+    )
     (pin "1")
     (pin "2")
@@
     )
     (property "Datasheet" "~" (at 203.2 58.42 0)
+      (effects (font (size 1.27 1.27)) hide)
+    )
+    (property "Farnell" "3013482" (at 203.2 58.42 0)
       (effects (font (size 1.27 1.27)) hide)
     )
@@
       (effects (font (size 1.27 1.27)) hide)
     )
+    (property "Farnell" "3013482" (at 95.25 78.74 0)
+      (effects (font (size 1.27 1.27)) hide)
+    )
     (pin "1")
     (pin "2")
@@
       (effects (font (size 1.27 1.27)))
     )
-    (property "Value" "L" (at 166.37 86.36 90)
-      (effects (font (size 1.27 1.27)))
-    )
-    (property "Footprint" "Inductor_SMD:L_0805_2012Metric" (at 166.37 88.9 0)
+    (property "Value" "0.5u" (at 166.37 86.36 90)
+      (effects (font (size 1.27 1.27)))
+    )
+    (property "Footprint" "Inductor_SMD:L_Bourns_SRN6045TA" (at 166.37 88.9 0)
       (effects (font (size 1.27 1.27)) hide)
     )
@@
       (effects (font (size 1.27 1.27)) hide)
     )
+    (property "Farnell" "3780754" (at 166.37 88.9 90)
+      (effects (font (size 1.27 1.27)) hide)
+    )

Commit message: - small (non functional) changes
Parts:
- C27: Farnell 2611943 -> 1867958
Other:
- note added: "Capacitor changed to: 1867958"
Changed lines of the file:
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@@
     (stroke (width 0) (type default))
+  )
+  (text "Capacitor changed to: 1867958" (at 162.56 121.92 90)
+    (effects (font (size 1.27 1.27)) (justify right bottom))
   )
   (label "AC.~{ENABLE}" (at 95.25 124.46 0) (fields_autoplaced)
@@
       (effects (font (size 1.27 1.27)) hide)
     )
-    (property "Farnell" "2611943" (at 156.21 111.76 0)
+    (property "Farnell" "1867958" (at 156.21 111.76 0)
       (effects (font (size 1.27 1.27)) hide)
     )
@@
       (effects (font (size 1.27 1.27)) hide)
     )
-    (property "Farnell" "2611943" (at 156.21 101.6 0)
+    (property "Farnell" "1867958" (at 156.21 101.6 0)
       (effects (font (size 1.27 1.27)) hide)
     )
@@
       (effects (font (size 1.27 1.27)) hide)
     )
-    (property "Farnell" "2611943" (at 156.21 121.92 0)
+    (property "Farnell" "1867958" (at 156.21 121.92 0)
       (effects (font (size 1.27 1.27)) hide)
     )
@@
       (effects (font (size 1.27 1.27)) hide)
     )
-    (property "Farnell" "2611943" (at 156.21 91.44 0)
-      (effects (font (size 1.27 1.27)) hide)
-    )
+    (property "Farnell" "1867958" (at 156.21 91.44 0)
+      (effects (font (size 1.27 1.27)) hide)
+    )
