File: pcb/I2STest.kicad_sch (KiCad schematic)
At the start: 8 parts, among them IC2 WM8804GEDS_V, J4 Conn_Coaxial, Y2 Crystal

Commit message: - voor aanpassing design rules jclpcb
Parts:
- C31, C32, C33: footprint (none) -> Capacitor_SMD:C_0805_2012Metric_Pad1.18x1.45mm_HandSolder
- R22, R23: footprint (none) -> Resistor_SMD:R_0805_2012Metric_Pad1.20x1.40mm_HandSolder
Changed lines of the file:
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@@
       (effects (font (size 1.27 1.27)) (justify left))
     )
-    (property "Footprint" "" (at 178.562 50.8 90)
+    (property "Footprint" "Resistor_SMD:R_0805_2012Metric_Pad1.20x1.40mm_HandSolder" (at 178.562 50.8 90)
       (effects (font (size 1.27 1.27)) hide)
     )
@@
       (effects (font (size 1.27 1.27)) (justify left))
     )
-    (property "Footprint" "" (at 171.1452 91.44 0)
+    (property "Footprint" "Capacitor_SMD:C_0805_2012Metric_Pad1.18x1.45mm_HandSolder" (at 171.1452 91.44 0)
       (effects (font (size 1.27 1.27)) hide)
     )
@@
       (effects (font (size 1.27 1.27)) (justify left))
     )
-    (property "Footprint" "" (at 155.9052 91.44 0)
+    (property "Footprint" "Capacitor_SMD:C_0805_2012Metric_Pad1.18x1.45mm_HandSolder" (at 155.9052 91.44 0)
       (effects (font (size 1.27 1.27)) hide)
     )
@@
       (effects (font (size 1.27 1.27)))
     )
-    (property "Footprint" "" (at 175.26 44.958 90)
+    (property "Footprint" "Resistor_SMD:R_0805_2012Metric_Pad1.20x1.40mm_HandSolder" (at 175.26 44.958 90)
       (effects (font (size 1.27 1.27)) hide)
     )
@@
       (effects (font (size 1.27 1.27)))
     )
-    (property "Footprint" "" (at 190.5 42.2148 0)
+    (property "Footprint" "Capacitor_SMD:C_0805_2012Metric_Pad1.18x1.45mm_HandSolder" (at 190.5 42.2148 0)
       (effects (font (size 1.27 1.27)) hide)
     )

Commit message: - cleanup ERC errors
Parts:
- J4: footprint (none) -> Connector_Coaxial:BNC_PanelMountable_Vertical
- Y2: value Crystal -> 12Mhz; footprint (none) -> Crystal:Crystal_SMD_Abracon_ABM3-2Pin_5.0x3.2mm_HandSoldering
Changed lines of the file:
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@@
   (no_connect (at 149.86 49.53))
   (no_connect (at 114.3 67.31))
-  (bus_entry (at 100.33 62.23) (size 2.54 2.54)
-    (stroke (width 0) (type default))
-  )
-  (bus_entry (at 100.33 59.69) (size 2.54 2.54)
-    (stroke (width 0) (type default))
-  )
-  (bus_entry (at 100.33 54.61) (size 2.54 2.54)
-    (stroke (width 0) (type default))
-  )
-  (bus_entry (at 100.33 57.15) (size 2.54 2.54)
+  (bus_entry (at 92.71 54.61) (size 2.54 2.54)
+    (stroke (width 0) (type default))
+  )
+  (bus_entry (at 92.71 62.23) (size 2.54 2.54)
+    (stroke (width 0) (type default))
+  )
+  (bus_entry (at 92.71 57.15) (size 2.54 2.54)
+    (stroke (width 0) (type default))
+  )
+  (bus_entry (at 92.71 59.69) (size 2.54 2.54)
     (stroke (width 0) (type default))
   )
@@
     (stroke (width 0) (type default))
   )
-  (bus (pts (xy 49.53 54.61) (xy 100.33 54.61))
-    (stroke (width 0) (type default))
-  )
-  (wire (pts (xy 102.87 64.77) (xy 114.3 64.77))
-    (stroke (width 0) (type default))
-  )
   (wire (pts (xy 111.76 36.83) (xy 111.76 38.1))
     (stroke (width 0) (type default))
   )
-  (bus (pts (xy 100.33 59.69) (xy 100.33 62.23))
-    (stroke (width 0) (type default))
-  )
   (wire (pts (xy 170.18 27.94) (xy 170.18 43.18))
     (stroke (width 0) (type default))
@@
     (stroke (width 0) (type default))
   )
-  (wire (pts (xy 102.87 59.69) (xy 114.3 59.69))
+  (wire (pts (xy 95.25 64.77) (xy 114.3 64.77))
     (stroke (width 0) (type default))
   )
@@
     (stroke (width 0) (type default))
   )
+  (bus (pts (xy 92.71 50.8) (xy 92.71 54.61))
+    (stroke (width 0) (type default))
+  )
   (wire (pts (xy 110.49 74.93) (xy 110.49 78.74))
     (stroke (width 0) (type default))
@@
     (stroke (width 0) (type default))
   )
-  (bus (pts (xy 100.33 54.61) (xy 100.33 57.15))
-    (stroke (width 0) (type default))
-  )
   (wire (pts (xy 110.49 74.93) (xy 114.3 74.93))
     (stroke (width 0) (type default))
   )
+  (wire (pts (xy 95.25 57.15) (xy 114.3 57.15))
+    (stroke (width 0) (type default))
+  )
   (wire (pts (xy 170.18 27.94) (xy 109.22 27.94))
     (stroke (width 0) (type default))
@@
     (stroke (width 0) (type default))
   )
+  (wire (pts (xy 95.25 59.69) (xy 114.3 59.69))
+    (stroke (width 0) (type default))
+  )
   (wire (pts (xy 111.76 41.91) (xy 114.3 41.91))
     (stroke (width 0) (type default))
@@
     (stroke (width 0) (type default))
   )
+  (wire (pts (xy 95.25 62.23) (xy 114.3 62.23))
+    (stroke (width 0) (type default))
+  )
   (wire (pts (xy 199.39 48.26) (xy 199.39 55.88))
     (stroke (width 0) (type default))
@@
     (stroke (width 0) (type default))
   )
-  (wire (pts (xy 102.87 57.15) (xy 114.3 57.15))
+  (bus (pts (xy 71.12 50.8) (xy 92.71 50.8))
     (stroke (width 0) (type default))
   )
@@
     (stroke (width 0) (type default))
   )
-  (bus (pts (xy 100.33 57.15) (xy 100.33 59.69))
-    (stroke (width 0) (type default))
-  )
   (wire (pts (xy 149.86 74.93) (xy 154.94 74.93))
     (stroke (width 0) (type default))
@@
     (stroke (width 0) (type default))
   )
-  (wire (pts (xy 102.87 62.23) (xy 114.3 62.23))
+  (bus (pts (xy 92.71 54.61) (xy 92.71 57.15))
     (stroke (width 0) (type default))
   )
@@
     (stroke (width 0) (type default))
   )
+  (bus (pts (xy 92.71 59.69) (xy 92.71 62.23))
+    (stroke (width 0) (type default))
+  )
   (wire (pts (xy 114.3 72.39) (xy 110.49 72.39))
     (stroke (width 0) (type default))
@@
     (stroke (width 0) (type default))
   )
+  (bus (pts (xy 92.71 57.15) (xy 92.71 59.69))
+    (stroke (width 0) (type default))
+  )
   (wire (pts (xy 111.76 38.1) (xy 111.76 41.91))
     (stroke (width 0) (type default))
@@
     (stroke (width 0) (type default))
   )
-  (label "I2S.BCK" (at 104.14 62.23 0)
+  (label "I2S.MCK" (at 99.06 57.15 0)
     (effects (font (size 1.27 1.27)) (justify left bottom))
   )
-  (label "I2S.MCK" (at 104.14 57.15 0)
+  (label "I2S.BCK" (at 99.06 62.23 0)
     (effects (font (size 1.27 1.27)) (justify left bottom))
   )
-  (label "I2S{LRCK BCK MCK D}" (at 58.42 54.61 0) (fields_autoplaced)
+  (label "I2S.LRCK" (at 99.06 59.69 0)
     (effects (font (size 1.27 1.27)) (justify left bottom))
   )
-  (label "I2S.D" (at 104.14 64.77 0)
+  (label "I2S.D" (at 99.06 64.77 0)
     (effects (font (size 1.27 1.27)) (justify left bottom))
   )
-  (label "I2S.LRCK" (at 104.14 59.69 0)
-    (effects (font (size 1.27 1.27)) (justify left bottom))
-  )
-  (hierarchical_label "I2S" (shape input) (at 49.53 54.61 180) (fields_autoplaced)
+  (hierarchical_label "I2S{LRCK BCK MCK D}" (shape input) (at 71.12 50.8 180) (fields_autoplaced)
     (effects (font (size 1.27 1.27)) (justify right))
   )
@@
         )
         (path "/c639bae0-d26f-43ee-9e8c-ca060284bd0b/434094c9-79fb-49fe-9eff-d35a4d1836d1"
-          (reference "#PWR031") (unit 1)
+          (reference "#PWR039") (unit 1)
         )
       )
@@
         )
         (path "/c639bae0-d26f-43ee-9e8c-ca060284bd0b/434094c9-79fb-49fe-9eff-d35a4d1836d1"
-          (reference "#PWR032") (unit 1)
+          (reference "#PWR040") (unit 1)
         )
       )
@@
       (effects (font (size 1.27 1.27)) (justify left))
     )
-    (property "Footprint" "" (at 199.39 43.18 0)
+    (property "Footprint" "Connector_Coaxial:BNC_PanelMountable_Vertical" (at 199.39 43.18 0)
       (effects (font (size 1.27 1.27)) hide)
     )
@@
         )
         (path "/c639bae0-d26f-43ee-9e8c-ca060284bd0b/434094c9-79fb-49fe-9eff-d35a4d1836d1"
-          (reference "J4") (unit 1)
+          (reference "J5") (unit 1)
         )
       )
@@
       (effects (font (size 1.27 1.27)))
     )
-    (property "Value" "Crystal" (at 161.29 87.63 0)
-      (effects (font (size 1.27 1.27)))
-    )
-    (property "Footprint" "" (at 162.56 81.28 0)
+    (property "Value" "12Mhz" (at 161.29 87.63 0)
+      (effects (font (size 1.27 1.27)))
+    )
+    (property "Footprint" "Crystal:Crystal_SMD_Abracon_ABM3-2Pin_5.0x3.2mm_HandSoldering" (at 162.56 81.28 0)
       (effects (font (size 1.27 1.27)) hide)
     )
@@
         )
         (path "/c639bae0-d26f-43ee-9e8c-ca060284bd0b/434094c9-79fb-49fe-9eff-d35a4d1836d1"
-          (reference "#PWR029") (unit 1)
+          (reference "#PWR037") (unit 1)
         )
       )
@@
         )
         (path "/c639bae0-d26f-43ee-9e8c-ca060284bd0b/434094c9-79fb-49fe-9eff-d35a4d1836d1"
-          (reference "C32") (unit 1)
+          (reference "C47") (unit 1)
         )
       )
@@
         )
         (path "/c639bae0-d26f-43ee-9e8c-ca060284bd0b/434094c9-79fb-49fe-9eff-d35a4d1836d1"
-          (reference "#PWR030") (unit 1)
+          (reference "#PWR038") (unit 1)
         )
       )
@@
         )
         (path "/c639bae0-d26f-43ee-9e8c-ca060284bd0b/434094c9-79fb-49fe-9eff-d35a4d1836d1"
-          (reference "C31") (unit 1)
+          (reference "C46") (unit 1)
         )
       )
@@
         )
         (path "/c639bae0-d26f-43ee-9e8c-ca060284bd0b/434094c9-79fb-49fe-9eff-d35a4d1836d1"
-          (reference "C33") (unit 1)
-        )
-      )
+          (reference "C48") (unit 1)
+        )
+      )

Commit message: - placing components
Parts:
- removed J4: Conn_Coaxial, Connector_Coaxial:BNC_PanelMountable_Vertical, symbol Connector:Conn_Coaxial
- added TP13 (x2): TestPoint, TestPoint:TestPoint_Bridge_Pitch2.54mm_Drill1.0mm, symbol Connector:TestPoint
Connections:
- net GND: now also TP13.1
- net at C33.2: now also TP13.1
Changed lines of the file:
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@@
   (junction (at 111.76 38.1) (diameter 0) (color 0 0 0 0)
   )
+  (junction (at 111.76 41.91) (diameter 0) (color 0 0 0 0)
+  )
   (junction (at 189.23 55.88) (diameter 0) (color 0 0 0 0)
-  )
-  (junction (at 111.76 41.91) (diameter 0) (color 0 0 0 0)
   )
   (junction (at 154.94 81.28) (diameter 0) (color 0 0 0 0)
@@
     (stroke (width 0) (type default))
   )
+  (wire (pts (xy 189.23 55.88) (xy 194.31 55.88))
+    (stroke (width 0) (type default))
+  )
   (wire (pts (xy 109.22 49.53) (xy 114.3 49.53))
     (stroke (width 0) (type default))
@@
     (stroke (width 0) (type default))
   )
-  (wire (pts (xy 199.39 48.26) (xy 199.39 55.88))
-    (stroke (width 0) (type default))
-  )
   (wire (pts (xy 162.56 91.44) (xy 162.56 92.71))
     (stroke (width 0) (type default))
   )
   (wire (pts (xy 109.22 27.94) (xy 109.22 49.53))
-    (stroke (width 0) (type default))
-  )
-  (wire (pts (xy 199.39 55.88) (xy 189.23 55.88))
     (stroke (width 0) (type default))
   )
@@
     )
   )
+  (symbol (lib_id "Connector:TestPoint") (at 194.31 55.88 270) (unit 1)
+    (in_bom yes) (on_board yes) (dnp no)
+    (property "Reference" "TP13" (at 198.247 57.785 0)
+      (effects (font (size 1.27 1.27)) (justify left))
+    )
+    (property "Value" "TestPoint" (at 195.707 57.785 0)
+      (effects (font (size 1.27 1.27)) (justify left))
+    )
+    (property "Footprint" "TestPoint:TestPoint_Bridge_Pitch2.54mm_Drill1.0mm" (at 194.31 60.96 0)
+      (effects (font (size 1.27 1.27)) hide)
+    )
+    (property "Datasheet" "" (at 194.31 60.96 0)
+      (effects (font (size 1.27 1.27)) hide)
+    )
+    (property "Field4" "nf" (at 194.31 55.88 0)
+      (effects (font (size 1.27 1.27)) hide)
+    )
+    (property "Field5" "nf" (at 194.31 55.88 0)
+      (effects (font (size 1.27 1.27)) hide)
+    )
+    (property "Field6" "nf" (at 194.31 55.88 0)
+      (effects (font (size 1.27 1.27)) hide)
+    )
+    (property "Field7" "nf" (at 194.31 55.88 0)
+      (effects (font (size 1.27 1.27)) hide)
+    )
+    (pin "1")
+    (instances
+      (project "VolumioAmp"
+        (path "/c639bae0-d26f-43ee-9e8c-ca060284bd0b/97b9f385-290b-4a5e-9fd5-e8b1b07223d1"
+          (reference "TP13") (unit 1)
+        )
+        (path "/c639bae0-d26f-43ee-9e8c-ca060284bd0b/434094c9-79fb-49fe-9eff-d35a4d1836d1"
+          (reference "TP22") (unit 1)
+        )
+      )
+      (project "CM4IOv5"
+        (path "/e63e39d7-6ac0-4ffd-8aa3-1841a4541b55/00000000-0000-0000-0000-00005d31f999"
+          (reference "TP4") (unit 1)
+        )
+      )
+    )
+  )
   (symbol (lib_id "power:GND") (at 189.23 55.88 0) (unit 1)
     (in_bom yes) (on_board yes) (dnp no)
@@
         (path "/e63e39d7-6ac0-4ffd-8aa3-1841a4541b55/00000000-0000-0000-0000-00005e072e02"
           (reference "#PWR013") (unit 1)
-        )
-      )
-    )
-  )
-  (symbol (lib_id "Connector:Conn_Coaxial") (at 199.39 43.18 0) (unit 1)
-    (in_bom yes) (on_board yes) (dnp no) (fields_autoplaced)
-    (property "Reference" "J4" (at 203.2 42.2032 0)
-      (effects (font (size 1.27 1.27)) (justify left))
-    )
-    (property "Value" "Conn_Coaxial" (at 203.2 44.7432 0)
-      (effects (font (size 1.27 1.27)) (justify left))
-    )
-    (property "Footprint" "Connector_Coaxial:BNC_PanelMountable_Vertical" (at 199.39 43.18 0)
-      (effects (font (size 1.27 1.27)) hide)
-    )
-    (property "Datasheet" " ~" (at 199.39 43.18 0)
-      (effects (font (size 1.27 1.27)) hide)
-    )
-    (pin "1")
-    (pin "2")
-    (instances
-      (project "VolumioAmp"
-        (path "/c639bae0-d26f-43ee-9e8c-ca060284bd0b/93301fd2-7a6d-48be-bd24-243a1877e343"
-          (reference "J4") (unit 1)
-        )
-        (path "/c639bae0-d26f-43ee-9e8c-ca060284bd0b/434094c9-79fb-49fe-9eff-d35a4d1836d1"
-          (reference "J5") (unit 1)
         )
       )
@@
         )
       )
+    )
+  )
+  (symbol (lib_id "Connector:TestPoint") (at 194.31 43.18 270) (unit 1)
+    (in_bom yes) (on_board yes) (dnp no)
+    (property "Reference" "TP13" (at 198.247 45.085 0)
+      (effects (font (size 1.27 1.27)) (justify left))
+    )
+    (property "Value" "TestPoint" (at 195.707 45.085 0)
+      (effects (font (size 1.27 1.27)) (justify left))
+    )
+    (property "Footprint" "TestPoint:TestPoint_Bridge_Pitch2.54mm_Drill1.0mm" (at 194.31 48.26 0)
+      (effects (font (size 1.27 1.27)) hide)
+    )
+    (property "Datasheet" "" (at 194.31 48.26 0)
+      (effects (font (size 1.27 1.27)) hide)
+    )
+    (property "Field4" "nf" (at 194.31 43.18 0)
+      (effects (font (size 1.27 1.27)) hide)
+    )
+    (property "Field5" "nf" (at 194.31 43.18 0)
+      (effects (font (size 1.27 1.27)) hide)
+    )
+    (property "Field6" "nf" (at 194.31 43.18 0)
+      (effects (font (size 1.27 1.27)) hide)
+    )
+    (property "Field7" "nf" (at 194.31 43.18 0)
+      (effects (font (size 1.27 1.27)) hide)
+    )
+    (pin "1")
+    (instances
+      (project "VolumioAmp"
+        (path "/c639bae0-d26f-43ee-9e8c-ca060284bd0b/97b9f385-290b-4a5e-9fd5-e8b1b07223d1"
+          (reference "TP13") (unit 1)
+        )
+        (path "/c639bae0-d26f-43ee-9e8c-ca060284bd0b/434094c9-79fb-49fe-9eff-d35a4d1836d1"
+          (reference "TP21") (unit 1)
+        )
+      )
+      (project "CM4IOv5"
+        (path "/e63e39d7-6ac0-4ffd-8aa3-1841a4541b55/00000000-0000-0000-0000-00005d31f999"
+          (reference "TP4") (unit 1)
+        )
+      )

Commit message: - component selection/place
Parts:
- TP13: footprint TestPoint:TestPoint_Bridge_Pitch2.54mm_Drill1.0mm -> TestPoint:TestPoint_Bridge_Pitch2.0mm_Drill0.7mm
Changed lines of the file:
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@@
         )
         (path "/c639bae0-d26f-43ee-9e8c-ca060284bd0b/434094c9-79fb-49fe-9eff-d35a4d1836d1"
-          (reference "#PWR040") (unit 1)
+          (reference "#PWR041") (unit 1)
         )
       )
@@
       (effects (font (size 1.27 1.27)) (justify left))
     )
-    (property "Footprint" "TestPoint:TestPoint_Bridge_Pitch2.54mm_Drill1.0mm" (at 194.31 60.96 0)
+    (property "Footprint" "TestPoint:TestPoint_Bridge_Pitch2.0mm_Drill0.7mm" (at 194.31 60.96 0)
       (effects (font (size 1.27 1.27)) hide)
     )
@@
         )
         (path "/c639bae0-d26f-43ee-9e8c-ca060284bd0b/434094c9-79fb-49fe-9eff-d35a4d1836d1"
-          (reference "TP22") (unit 1)
+          (reference "TP25") (unit 1)
         )
       )
@@
         )
         (path "/c639bae0-d26f-43ee-9e8c-ca060284bd0b/434094c9-79fb-49fe-9eff-d35a4d1836d1"
-          (reference "#PWR041") (unit 1)
+          (reference "#PWR042") (unit 1)
         )
       )
@@
         )
         (path "/c639bae0-d26f-43ee-9e8c-ca060284bd0b/434094c9-79fb-49fe-9eff-d35a4d1836d1"
-          (reference "R23") (unit 1)
+          (reference "R24") (unit 1)
         )
       )
@@
         )
         (path "/c639bae0-d26f-43ee-9e8c-ca060284bd0b/434094c9-79fb-49fe-9eff-d35a4d1836d1"
-          (reference "#PWR038") (unit 1)
+          (reference "#PWR039") (unit 1)
         )
       )
@@
         )
         (path "/c639bae0-d26f-43ee-9e8c-ca060284bd0b/434094c9-79fb-49fe-9eff-d35a4d1836d1"
-          (reference "C47") (unit 1)
+          (reference "C50") (unit 1)
         )
       )
@@
         )
         (path "/c639bae0-d26f-43ee-9e8c-ca060284bd0b/434094c9-79fb-49fe-9eff-d35a4d1836d1"
-          (reference "#PWR039") (unit 1)
+          (reference "#PWR040") (unit 1)
         )
       )
@@
       (effects (font (size 1.27 1.27)) (justify left))
     )
-    (property "Footprint" "TestPoint:TestPoint_Bridge_Pitch2.54mm_Drill1.0mm" (at 194.31 48.26 0)
+    (property "Footprint" "TestPoint:TestPoint_Bridge_Pitch2.0mm_Drill0.7mm" (at 194.31 48.26 0)
       (effects (font (size 1.27 1.27)) hide)
     )
@@
         )
         (path "/c639bae0-d26f-43ee-9e8c-ca060284bd0b/434094c9-79fb-49fe-9eff-d35a4d1836d1"
-          (reference "TP21") (unit 1)
+          (reference "TP24") (unit 1)
         )
       )
@@
         )
         (path "/c639bae0-d26f-43ee-9e8c-ca060284bd0b/434094c9-79fb-49fe-9eff-d35a4d1836d1"
-          (reference "C46") (unit 1)
+          (reference "C49") (unit 1)
         )
       )
@@
         )
         (path "/c639bae0-d26f-43ee-9e8c-ca060284bd0b/434094c9-79fb-49fe-9eff-d35a4d1836d1"
-          (reference "R22") (unit 1)
+          (reference "R23") (unit 1)
         )
       )
@@
         )
         (path "/c639bae0-d26f-43ee-9e8c-ca060284bd0b/434094c9-79fb-49fe-9eff-d35a4d1836d1"
-          (reference "C48") (unit 1)
-        )
-      )
+          (reference "C51") (unit 1)
+        )
+      )
