File: pcb/I2STest.kicad_sch (KiCad schematic)
At the start: 9 parts, among them IC2 WM8804GEDS_V, Y2 12Mhz

Commit message: - BOM added (Farnell nrs)
Parts:
- C31, C32: value 22n -> 22p; Farnell (none) -> 2896721
- C33: value C -> 1u; Farnell (none) -> 3013482
- R22: value R -> 210R; Farnell (none) -> 2326770
- R23: value R -> 110R; Farnell (none) -> 1894172
- Y2: Farnell (none) -> 2101327
Changed lines of the file:
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@@
+      (effects (font (size 1.27 1.27)) hide)
+    )
+    (property "Farnell" "2101327" (at 162.56 81.28 0)
       (effects (font (size 1.27 1.27)) hide)
     )
@@
       (effects (font (size 1.27 1.27)) (justify left))
     )
-    (property "Value" "R" (at 182.88 52.07 0)
+    (property "Value" "110R" (at 182.88 52.07 0)
       (effects (font (size 1.27 1.27)) (justify left))
     )
@@
     )
     (property "Datasheet" "~" (at 180.34 50.8 0)
+      (effects (font (size 1.27 1.27)) hide)
+    )
+    (property "Farnell" "1894172" (at 180.34 50.8 0)
       (effects (font (size 1.27 1.27)) hide)
     )
@@
       (effects (font (size 1.27 1.27)) (justify left))
     )
-    (property "Value" "22n" (at 173.99 88.9 0)
+    (property "Value" "22p" (at 173.99 88.9 0)
       (effects (font (size 1.27 1.27)) (justify left))
     )
@@
     )
     (property "Datasheet" "~" (at 170.18 87.63 0)
+      (effects (font (size 1.27 1.27)) hide)
+    )
+    (property "Farnell" "2896721" (at 170.18 87.63 0)
       (effects (font (size 1.27 1.27)) hide)
     )
@@
       (effects (font (size 1.27 1.27)) (justify left))
     )
-    (property "Value" "22n" (at 148.59 88.9 0)
+    (property "Value" "22p" (at 148.59 88.9 0)
       (effects (font (size 1.27 1.27)) (justify left))
     )
@@
     )
     (property "Datasheet" "~" (at 154.94 87.63 0)
+      (effects (font (size 1.27 1.27)) hide)
+    )
+    (property "Farnell" "2896721" (at 154.94 87.63 0)
       (effects (font (size 1.27 1.27)) hide)
     )
@@
       (effects (font (size 1.27 1.27)))
     )
-    (property "Value" "R" (at 175.26 39.37 90)
+    (property "Value" "210R" (at 175.26 39.37 90)
       (effects (font (size 1.27 1.27)))
     )
@@
     )
     (property "Datasheet" "~" (at 175.26 43.18 0)
+      (effects (font (size 1.27 1.27)) hide)
+    )
+    (property "Farnell" "2326770" (at 175.26 43.18 0)
       (effects (font (size 1.27 1.27)) hide)
     )
@@
       (effects (font (size 1.27 1.27)))
     )
-    (property "Value" "C" (at 186.69 38.1 90)
+    (property "Value" "1u" (at 186.69 38.1 90)
       (effects (font (size 1.27 1.27)))
     )
@@
       (effects (font (size 1.27 1.27)) hide)
     )
+    (property "Farnell" "3013482" (at 186.69 43.18 0)
+      (effects (font (size 1.27 1.27)) hide)
+    )
