File: pcb/CM4_Ethernet.kicad_sch (KiCad schematic)
At the start: 18 parts, among them J1 L829-1J1T-43, U1 74LVC1G07SE-7, U1 TPD4EUSB30, U2 TPD4EUSB30

Commit message: - component selection/place
Parts:
- added TP1, TP3: TestPoint, TestPoint:TestPoint_Bridge_Pitch2.54mm_Drill1.0mm, symbol Connector:TestPoint
- TP4: renamed from TP1; footprint TestPoint:TestPoint_Bridge_Pitch2.54mm_Drill1.0mm -> TestPoint:TestPoint_THTPad_1.0x1.0mm_Drill0.5mm
Connections:
- net at D2.1 (K), R3.1: no longer TP2.1
- net at Module1.92 (RUN_PG): now also TP1.1
- net at Module1.93 (nRPIBOOT): now also TP2.1
- net at Module1.99 (Global_EN): now also TP3.1
- no-connect marks 46 -> 43
Changed lines of the file:
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@@
   (junction (at 50.8 36.83) (diameter 1.016) (color 0 0 0 0)
-  )
-  (junction (at 165.1 133.35) (diameter 1.016) (color 0 0 0 0)
   )
   (junction (at 114.3 44.45) (diameter 1.016) (color 0 0 0 0)
@@
   (no_connect (at 38.1 95.25))
   (no_connect (at 52.07 105.41))
-  (no_connect (at 52.07 143.51))
   (no_connect (at 113.03 107.95))
   (no_connect (at 127 80.01))
@@
   (no_connect (at 38.1 77.47))
   (no_connect (at 52.07 146.05))
-  (no_connect (at 113.03 146.05))
   (no_connect (at 127 97.79))
   (no_connect (at 52.07 52.07))
   (no_connect (at 113.03 120.65))
-  (no_connect (at 113.03 153.67))
   (no_connect (at 52.07 115.57))
   (no_connect (at 127 92.71))
@@
     (stroke (width 0) (type solid))
   )
+  (wire (pts (xy 44.45 143.51) (xy 52.07 143.51))
+    (stroke (width 0) (type default))
+  )
   (wire (pts (xy 203.2 38.1) (xy 210.82 38.1))
     (stroke (width 0) (type solid))
@@
     (stroke (width 0) (type default))
   )
+  (wire (pts (xy 120.65 146.05) (xy 120.65 144.78))
+    (stroke (width 0) (type default))
+  )
   (wire (pts (xy 129.54 41.91) (xy 129.54 39.37))
     (stroke (width 0) (type solid))
@@
     (stroke (width 0) (type solid))
   )
-  (wire (pts (xy 160.02 133.35) (xy 165.1 133.35))
-    (stroke (width 0) (type solid))
-  )
   (wire (pts (xy 218.44 63.5) (xy 218.44 62.23))
     (stroke (width 0) (type default))
@@
     (stroke (width 0) (type solid))
   )
+  (wire (pts (xy 113.03 153.67) (xy 123.19 153.67))
+    (stroke (width 0) (type default))
+  )
   (wire (pts (xy 236.22 90.17) (xy 243.84 90.17))
     (stroke (width 0) (type solid))
@@
   (wire (pts (xy 114.3 95.25) (xy 114.3 102.87))
     (stroke (width 0) (type solid))
+  )
+  (wire (pts (xy 113.03 146.05) (xy 120.65 146.05))
+    (stroke (width 0) (type default))
   )
   (wire (pts (xy 218.44 100.33) (xy 243.84 100.33))
@@
         )
         (path "/c639bae0-d26f-43ee-9e8c-ca060284bd0b/0d83f7c4-6343-47e0-83de-c41ded3b9d5e"
-          (reference "R4") (unit 1)
+          (reference "R5") (unit 1)
         )
       )
@@
     )
   )
-  (symbol (lib_id "Connector:TestPoint") (at 160.02 133.35 90) (unit 1)
-    (in_bom yes) (on_board yes) (dnp no)
-    (property "Reference" "TP2" (at 157.6578 130.683 90)
+  (symbol (lib_id "Connector:TestPoint") (at 120.65 144.78 0) (unit 1)
+    (in_bom yes) (on_board yes) (dnp no)
+    (property "Reference" "TP2" (at 124.46 143.51 90)
       (effects (font (size 1.27 1.27)) (justify left))
     )
-    (property "Value" "TestPoint" (at 162.7378 135.763 90)
+    (property "Value" "TestPoint" (at 122.555 146.05 90)
       (effects (font (size 1.27 1.27)) (justify left))
     )
-    (property "Footprint" "TestPoint:TestPoint_Bridge_Pitch2.54mm_Drill1.0mm" (at 160.02 128.27 0)
-      (effects (font (size 1.27 1.27)) hide)
-    )
-    (property "Datasheet" "" (at 160.02 128.27 0)
-      (effects (font (size 1.27 1.27)) hide)
-    )
-    (property "Field4" "nf" (at 160.02 133.35 0)
-      (effects (font (size 1.27 1.27)) hide)
-    )
-    (property "Field5" "nf" (at 160.02 133.35 0)
-      (effects (font (size 1.27 1.27)) hide)
-    )
-    (property "Field6" "nf" (at 160.02 133.35 0)
-      (effects (font (size 1.27 1.27)) hide)
-    )
-    (property "Field7" "nf" (at 160.02 133.35 0)
+    (property "Footprint" "TestPoint:TestPoint_Bridge_Pitch2.54mm_Drill1.0mm" (at 125.73 144.78 0)
+      (effects (font (size 1.27 1.27)) hide)
+    )
+    (property "Datasheet" "" (at 125.73 144.78 0)
+      (effects (font (size 1.27 1.27)) hide)
+    )
+    (property "Field4" "nf" (at 120.65 144.78 0)
+      (effects (font (size 1.27 1.27)) hide)
+    )
+    (property "Field5" "nf" (at 120.65 144.78 0)
+      (effects (font (size 1.27 1.27)) hide)
+    )
+    (property "Field6" "nf" (at 120.65 144.78 0)
+      (effects (font (size 1.27 1.27)) hide)
+    )
+    (property "Field7" "nf" (at 120.65 144.78 0)
       (effects (font (size 1.27 1.27)) hide)
     )
@@
       (project "CM4IOv5"
         (path "/e63e39d7-6ac0-4ffd-8aa3-1841a4541b55/00000000-0000-0000-0000-00005cff706a"
-          (reference "TP5") (unit 1)
+          (reference "TP3") (unit 1)
         )
       )
@@
         (path "/e63e39d7-6ac0-4ffd-8aa3-1841a4541b55/00000000-0000-0000-0000-00005cff706a"
           (reference "#PWR05") (unit 1)
+        )
+      )
+    )
+  )
+  (symbol (lib_id "Connector:TestPoint") (at 44.45 143.51 90) (unit 1)
+    (in_bom yes) (on_board yes) (dnp no)
+    (property "Reference" "TP1" (at 43.18 139.7 90)
+      (effects (font (size 1.27 1.27)) (justify left))
+    )
+    (property "Value" "TestPoint" (at 45.72 141.605 90)
+      (effects (font (size 1.27 1.27)) (justify left))
+    )
+    (property "Footprint" "TestPoint:TestPoint_Bridge_Pitch2.54mm_Drill1.0mm" (at 44.45 138.43 0)
+      (effects (font (size 1.27 1.27)) hide)
+    )
+    (property "Datasheet" "" (at 44.45 138.43 0)
+      (effects (font (size 1.27 1.27)) hide)
+    )
+    (property "Field4" "nf" (at 44.45 143.51 0)
+      (effects (font (size 1.27 1.27)) hide)
+    )
+    (property "Field5" "nf" (at 44.45 143.51 0)
+      (effects (font (size 1.27 1.27)) hide)
+    )
+    (property "Field6" "nf" (at 44.45 143.51 0)
+      (effects (font (size 1.27 1.27)) hide)
+    )
+    (property "Field7" "nf" (at 44.45 143.51 0)
+      (effects (font (size 1.27 1.27)) hide)
+    )
+    (pin "1")
+    (instances
+      (project "VolumioAmp"
+        (path "/c639bae0-d26f-43ee-9e8c-ca060284bd0b/0d83f7c4-6343-47e0-83de-c41ded3b9d5e"
+          (reference "TP1") (unit 1)
+        )
+      )
+      (project "CM4IOv5"
+        (path "/e63e39d7-6ac0-4ffd-8aa3-1841a4541b55/00000000-0000-0000-0000-00005cff706a"
+          (reference "TP3") (unit 1)
         )
       )
@@
         )
         (path "/c639bae0-d26f-43ee-9e8c-ca060284bd0b/0d83f7c4-6343-47e0-83de-c41ded3b9d5e"
-          (reference "R24") (unit 1)
+          (reference "R4") (unit 1)
         )
       )
@@
         (path "/e63e39d7-6ac0-4ffd-8aa3-1841a4541b55/00000000-0000-0000-0000-00005cff706a"
           (reference "R2") (unit 1)
+        )
+      )
+    )
+  )
+  (symbol (lib_id "Connector:TestPoint") (at 123.19 153.67 270) (unit 1)
+    (in_bom yes) (on_board yes) (dnp no)
+    (property "Reference" "TP3" (at 124.46 157.48 90)
+      (effects (font (size 1.27 1.27)) (justify left))
+    )
+    (property "Value" "TestPoint" (at 121.92 155.575 90)
+      (effects (font (size 1.27 1.27)) (justify left))
+    )
+    (property "Footprint" "TestPoint:TestPoint_Bridge_Pitch2.54mm_Drill1.0mm" (at 123.19 158.75 0)
+      (effects (font (size 1.27 1.27)) hide)
+    )
+    (property "Datasheet" "" (at 123.19 158.75 0)
+      (effects (font (size 1.27 1.27)) hide)
+    )
+    (property "Field4" "nf" (at 123.19 153.67 0)
+      (effects (font (size 1.27 1.27)) hide)
+    )
+    (property "Field5" "nf" (at 123.19 153.67 0)
+      (effects (font (size 1.27 1.27)) hide)
+    )
+    (property "Field6" "nf" (at 123.19 153.67 0)
+      (effects (font (size 1.27 1.27)) hide)
+    )
+    (property "Field7" "nf" (at 123.19 153.67 0)
+      (effects (font (size 1.27 1.27)) hide)
+    )
+    (pin "1")
+    (instances
+      (project "VolumioAmp"
+        (path "/c639bae0-d26f-43ee-9e8c-ca060284bd0b/0d83f7c4-6343-47e0-83de-c41ded3b9d5e"
+          (reference "TP3") (unit 1)
+        )
+      )
+      (project "CM4IOv5"
+        (path "/e63e39d7-6ac0-4ffd-8aa3-1841a4541b55/00000000-0000-0000-0000-00005cff706a"
+          (reference "TP3") (unit 1)
         )
       )
@@
   (symbol (lib_id "Connector:TestPoint") (at 135.89 41.91 270) (unit 1)
     (in_bom yes) (on_board yes) (dnp no)
-    (property "Reference" "TP1" (at 137.16 45.72 90)
+    (property "Reference" "TP4" (at 137.16 45.72 90)
       (effects (font (size 1.27 1.27)) (justify left))
     )
@@
       (effects (font (size 1.27 1.27)) (justify left))
     )
-    (property "Footprint" "TestPoint:TestPoint_Bridge_Pitch2.54mm_Drill1.0mm" (at 135.89 46.99 0)
+    (property "Footprint" "TestPoint:TestPoint_THTPad_1.0x1.0mm_Drill0.5mm" (at 135.89 46.99 0)
       (effects (font (size 1.27 1.27)) hide)
     )
@@
       (project "VolumioAmp"
         (path "/c639bae0-d26f-43ee-9e8c-ca060284bd0b/0d83f7c4-6343-47e0-83de-c41ded3b9d5e"
-          (reference "TP1") (unit 1)
+          (reference "TP4") (unit 1)
         )
       )
@@
         )
         (path "/c639bae0-d26f-43ee-9e8c-ca060284bd0b/0d83f7c4-6343-47e0-83de-c41ded3b9d5e"
-          (reference "R5") (unit 1)
-        )
-      )
+          (reference "R6") (unit 1)
+        )
+      )

Commit message: - wiring
Parts:
- TP1, TP2, TP3: footprint TestPoint:TestPoint_Bridge_Pitch2.54mm_Drill1.0mm -> TestPoint:TestPoint_THTPad_1.0x1.0mm_Drill0.5mm
Changed lines of the file:
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@@
       (effects (font (size 1.27 1.27)) (justify left))
     )
-    (property "Footprint" "TestPoint:TestPoint_Bridge_Pitch2.54mm_Drill1.0mm" (at 125.73 144.78 0)
+    (property "Footprint" "TestPoint:TestPoint_THTPad_1.0x1.0mm_Drill0.5mm" (at 125.73 144.78 0)
       (effects (font (size 1.27 1.27)) hide)
     )
@@
       (effects (font (size 1.27 1.27)) (justify left))
     )
-    (property "Footprint" "TestPoint:TestPoint_Bridge_Pitch2.54mm_Drill1.0mm" (at 44.45 138.43 0)
+    (property "Footprint" "TestPoint:TestPoint_THTPad_1.0x1.0mm_Drill0.5mm" (at 44.45 138.43 0)
       (effects (font (size 1.27 1.27)) hide)
     )
@@
       (effects (font (size 1.27 1.27)) (justify left))
     )
-    (property "Footprint" "TestPoint:TestPoint_Bridge_Pitch2.54mm_Drill1.0mm" (at 123.19 158.75 0)
-      (effects (font (size 1.27 1.27)) hide)
-    )
+    (property "Footprint" "TestPoint:TestPoint_THTPad_1.0x1.0mm_Drill0.5mm" (at 123.19 158.75 0)
+      (effects (font (size 1.27 1.27)) hide)
+    )

Commit message: - BOM added (Farnell nrs)
Parts:
- C1: footprint Capacitor_SMD:C_0402_1005Metric -> Capacitor_SMD:C_01005_0402Metric; Farnell (none) -> 2409031; Field5 2611911 -> 2409031
- D1, D2: Farnell (none) -> 2991544
- R1, R2: Farnell (none) -> 2861091
- R2, R3: Farnell (none) -> 3546693
- U1: Farnell (none) -> 1845213
- U1, U2: Farnell (none) -> 3116518
Changed lines of the file:
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@@
+      (effects (font (size 1.27 1.27)) hide)
+    )
+    (property "Farnell" "3116518" (at 190.5 72.39 0)
       (effects (font (size 1.27 1.27)) hide)
     )
@@
       (effects (font (size 1.27 1.27)) hide)
     )
+    (property "Farnell" "3546693" (at 129.54 48.26 0)
+      (effects (font (size 1.27 1.27)) hide)
+    )
     (pin "1")
     (pin "2")
@@
       (effects (font (size 1.27 1.27)) hide)
     )
+    (property "Farnell" "2991544" (at 165.1 129.54 0)
+      (effects (font (size 1.27 1.27)) hide)
+    )
     (pin "1")
     (pin "2")
@@
     )
     (property "Part Description" "Buffer, Non-Inverting 1 Element 1 Bit per Element Open Drain Output SOT-353" (at 157.48 148.59 0)
+      (effects (font (size 1.27 1.27)) hide)
+    )
+    (property "Farnell" "1845213" (at 157.48 148.59 0)
       (effects (font (size 1.27 1.27)) hide)
     )
@@
     )
     (property "Part Description" "Resistor 470R M1005 1% 63mW" (at 214.63 100.33 0)
+      (effects (font (size 1.27 1.27)) hide)
+    )
+    (property "Farnell" "2861091" (at 214.63 100.33 0)
       (effects (font (size 1.27 1.27)) hide)
     )
@@
       (effects (font (size 1.27 1.27)) hide)
     )
+    (property "Farnell" "2991544" (at 129.54 35.56 0)
+      (effects (font (size 1.27 1.27)) hide)
+    )
     (pin "1")
     (pin "2")
@@
       (effects (font (size 1.27 1.27)) (justify left))
     )
-    (property "Footprint" "Capacitor_SMD:C_0402_1005Metric" (at 219.4052 62.23 0)
+    (property "Footprint" "Capacitor_SMD:C_01005_0402Metric" (at 219.4052 62.23 0)
       (effects (font (size 1.27 1.27)) hide)
     )
@@
       (effects (font (size 1.27 1.27)) hide)
     )
-    (property "Field5" "2611911" (at 218.44 58.42 0)
+    (property "Field5" "2409031" (at 218.44 58.42 0)
       (effects (font (size 1.27 1.27)) hide)
     )
@@
     )
     (property "Field8" "110091611" (at 218.44 58.42 0)
+      (effects (font (size 1.27 1.27)) hide)
+    )
+    (property "Farnell" "2409031" (at 218.44 58.42 0)
       (effects (font (size 1.27 1.27)) hide)
     )
@@
     )
     (property "Part Description" "Resistor 470R M1005 1% 63mW" (at 214.63 93.98 0)
+      (effects (font (size 1.27 1.27)) hide)
+    )
+    (property "Farnell" "2861091" (at 214.63 93.98 0)
       (effects (font (size 1.27 1.27)) hide)
     )
@@
       (effects (font (size 1.27 1.27)) hide)
     )
+    (property "Farnell" "3116518" (at 190.5 40.64 0)
+      (effects (font (size 1.27 1.27)) hide)
+    )
     (pin "1")
     (pin "10")
@@
       (effects (font (size 1.27 1.27)) hide)
     )
+    (property "Farnell" "2861091" (at 215.9 85.09 0)
+      (effects (font (size 1.27 1.27)) hide)
+    )
     (pin "1")
     (pin "2")
@@
       (effects (font (size 1.27 1.27)) hide)
     )
+    (property "Farnell" "3546693" (at 165.1 138.43 0)
+      (effects (font (size 1.27 1.27)) hide)
+    )
