File: pcb/CM4_HighSpeed.kicad_sch (KiCad schematic)
At the start: 2 parts

Commit message: - USB sound wired
Parts:
- renumbered R13 to R1
Changed lines of the file:
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@@
   (symbol (lib_id "Device:R") (at 153.67 45.72 0) (unit 1)
     (in_bom yes) (on_board yes) (dnp no)
-    (property "Reference" "R13" (at 147.955 44.45 0)
+    (property "Reference" "R1" (at 147.955 44.45 0)
       (effects (font (size 1.27 1.27)) (justify left))
     )
@@
       (project "VolumioAmp"
         (path "/c639bae0-d26f-43ee-9e8c-ca060284bd0b/714de229-102b-48b6-a22b-2290164179cf"
-          (reference "R13") (unit 1)
+          (reference "R1") (unit 1)
         )
       )
@@
   (symbol (lib_id "power:GND") (at 133.35 166.37 0) (unit 1)
     (in_bom yes) (on_board yes) (dnp no)
-    (property "Reference" "#PWR08" (at 133.35 172.72 0)
+    (property "Reference" "#PWR02" (at 133.35 172.72 0)
       (effects (font (size 1.27 1.27)) hide)
     )
@@
       (project "VolumioAmp"
         (path "/c639bae0-d26f-43ee-9e8c-ca060284bd0b/714de229-102b-48b6-a22b-2290164179cf"
-          (reference "#PWR08") (unit 1)
+          (reference "#PWR02") (unit 1)
         )
       )
@@
   (symbol (lib_id "power:GND") (at 153.67 49.53 0) (unit 1)
     (in_bom yes) (on_board yes) (dnp no)
-    (property "Reference" "#PWR022" (at 153.67 55.88 0)
+    (property "Reference" "#PWR03" (at 153.67 55.88 0)
       (effects (font (size 1.27 1.27)) hide)
     )
@@
       (project "VolumioAmp"
         (path "/c639bae0-d26f-43ee-9e8c-ca060284bd0b/714de229-102b-48b6-a22b-2290164179cf"
-          (reference "#PWR022") (unit 1)
+          (reference "#PWR03") (unit 1)
         )
       )
@@
   (symbol (lib_id "power:GND") (at 67.31 166.37 0) (unit 1)
     (in_bom yes) (on_board yes) (dnp no)
-    (property "Reference" "#PWR07" (at 67.31 172.72 0)
+    (property "Reference" "#PWR01" (at 67.31 172.72 0)
       (effects (font (size 1.27 1.27)) hide)
     )
@@
       (project "VolumioAmp"
         (path "/c639bae0-d26f-43ee-9e8c-ca060284bd0b/714de229-102b-48b6-a22b-2290164179cf"
-          (reference "#PWR07") (unit 1)
+          (reference "#PWR01") (unit 1)
         )
       )

Commit message: - voor aanpassing design rules jclpcb
Parts:
- R1: footprint Resistor_SMD:R_0402_1005Metric -> Resistor_SMD:R_0805_2012Metric_Pad1.20x1.40mm_HandSolder
Changed lines of the file:
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@@
       (effects (font (size 1.27 1.27)) (justify left))
     )
-    (property "Footprint" "Resistor_SMD:R_0402_1005Metric" (at 151.892 45.72 90)
+    (property "Footprint" "Resistor_SMD:R_0805_2012Metric_Pad1.20x1.40mm_HandSolder" (at 151.892 45.72 90)
       (effects (font (size 1.27 1.27)) hide)
     )

Commit message: - cleanup ERC errors
Parts:
- Module1: footprint CM4IO:Raspberry-Pi-4-Compute-Module -> Footprints:Raspberry-Pi-4-Compute-Module
Changed lines of the file:
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@@
       (effects (font (size 1.27 1.27)))
     )
-    (property "Footprint" "CM4IO:Raspberry-Pi-4-Compute-Module" (at 102.87 123.19 0)
+    (property "Footprint" "Footprints:Raspberry-Pi-4-Compute-Module" (at 102.87 123.19 0)
       (effects (font (size 1.27 1.27)) hide)
     )

Commit message: - ERC checks
Parts:
- Module1: footprint Footprints:Raspberry-Pi-4-Compute-Module -> CM4IO:Raspberry-Pi-4-Compute-Module; Field5 2off DF40C-100DS-0.4V -> 2x DF40C-100DS-0.4V
Changed lines of the file:
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@@
       (effects (font (size 1.27 1.27)))
     )
-    (property "Footprint" "Footprints:Raspberry-Pi-4-Compute-Module" (at 102.87 123.19 0)
+    (property "Footprint" "CM4IO:Raspberry-Pi-4-Compute-Module" (at 102.87 123.19 0)
       (effects (font (size 1.27 1.27)) hide)
     )
@@
       (effects (font (size 1.27 1.27)))
     )
-    (property "Field5" "2off DF40C-100DS-0.4V" (at 100.33 31.1658 0)
+    (property "Field5" "2x DF40C-100DS-0.4V" (at 100.33 31.1658 0)
       (effects (font (size 1.27 1.27)))
     )
@@
     )
   )
-  (symbol (lib_id "power:GND") (at 153.67 49.53 0) (unit 1)
+  (symbol (lib_name "GND_1") (lib_id "power:GND") (at 153.67 49.53 0) (unit 1)
     (in_bom yes) (on_board yes) (dnp no)
     (property "Reference" "#PWR03" (at 153.67 55.88 0)
@@
     )
   )
-  (symbol (lib_id "power:GND") (at 67.31 166.37 0) (unit 1)
+  (symbol (lib_name "GND_2") (lib_id "power:GND") (at 67.31 166.37 0) (unit 1)
     (in_bom yes) (on_board yes) (dnp no)
     (property "Reference" "#PWR01" (at 67.31 172.72 0)

Commit message: - work in progress, changed rj45 connector
Parts:
- Module1: footprint CM4IO:Raspberry-Pi-4-Compute-Module -> Footprints:Raspberry-Pi-4-Compute-Module
Changed lines of the file:
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@@
       (effects (font (size 1.27 1.27)))
     )
-    (property "Footprint" "CM4IO:Raspberry-Pi-4-Compute-Module" (at 102.87 123.19 0)
+    (property "Footprint" "Footprints:Raspberry-Pi-4-Compute-Module" (at 102.87 123.19 0)
       (effects (font (size 1.27 1.27)) hide)
     )

Commit message: - placing components
Parts:
- Module1: Farnell (none) -> 2427679
Changed lines of the file:
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@@
+      (effects (font (size 1.27 1.27)) hide)
+    )
+    (property "Farnell" "2427679" (at -39.37 96.52 0)
       (effects (font (size 1.27 1.27)) hide)
     )

Commit message: - BOM added (Farnell nrs)
Parts:
- R1: Farnell (none) -> 1576464
Changed lines of the file:
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@@
+      (effects (font (size 1.27 1.27)) hide)
+    )
+    (property "Farnell" "1576464" (at 153.67 45.72 0)
       (effects (font (size 1.27 1.27)) hide)
     )
