File: pcb/Power.kicad_sch (KiCad schematic)
At the start: 35 parts, among them J3 24v Input, Q1 DMP3013SFV-7, U6 AP64501SP-13, U7 LT1761-3.3

Commit message: - routed
Parts:
- renumbered TP15 to TP14, TP16 to TP15, TP17 to TP16
Changed lines of the file:
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@@
   (symbol (lib_id "Connector:TestPoint") (at 172.72 111.76 0) (unit 1)
     (in_bom yes) (on_board yes) (dnp no)
-    (property "Reference" "TP16" (at 174.625 107.823 0)
+    (property "Reference" "TP15" (at 174.625 107.823 0)
       (effects (font (size 1.27 1.27)) (justify left))
     )
@@
       (project "VolumioAmp"
         (path "/c639bae0-d26f-43ee-9e8c-ca060284bd0b/97b9f385-290b-4a5e-9fd5-e8b1b07223d1"
-          (reference "TP16") (unit 1)
+          (reference "TP15") (unit 1)
         )
       )
@@
   (symbol (lib_id "Connector:TestPoint") (at 110.49 38.1 0) (unit 1)
     (in_bom yes) (on_board yes) (dnp no)
-    (property "Reference" "TP15" (at 111.9632 35.1028 0)
+    (property "Reference" "TP14" (at 111.9632 35.1028 0)
       (effects (font (size 1.27 1.27)) (justify left))
     )
@@
       (project "VolumioAmp"
         (path "/c639bae0-d26f-43ee-9e8c-ca060284bd0b/97b9f385-290b-4a5e-9fd5-e8b1b07223d1"
-          (reference "TP15") (unit 1)
+          (reference "TP14") (unit 1)
         )
       )
@@
   (symbol (lib_id "Connector:TestPoint") (at 191.77 134.62 0) (unit 1)
     (in_bom yes) (on_board yes) (dnp no)
-    (property "Reference" "TP17" (at 193.2432 131.6228 0)
+    (property "Reference" "TP16" (at 193.2432 131.6228 0)
       (effects (font (size 1.27 1.27)) (justify left))
     )
@@
       (project "VolumioAmp"
         (path "/c639bae0-d26f-43ee-9e8c-ca060284bd0b/97b9f385-290b-4a5e-9fd5-e8b1b07223d1"
-          (reference "TP17") (unit 1)
-        )
-      )
+          (reference "TP16") (unit 1)
+        )
+      )

Commit message: - routed
Changed lines of the file:
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@@
   (junction (at 71.12 53.34) (diameter 1.016) (color 0 0 0 0)
   )
+  (junction (at 228.6 52.07) (diameter 0) (color 0 0 0 0)
+  )
   (junction (at 163.83 128.27) (diameter 1.016) (color 0 0 0 0)
   )
@@
   (junction (at 59.69 133.35) (diameter 1.016) (color 0 0 0 0)
   )
-  (junction (at 228.6 52.07) (diameter 0) (color 0 0 0 0)
-  )
   (junction (at 143.51 128.27) (diameter 1.016) (color 0 0 0 0)
   )
@@
     (stroke (width 0) (type default))
   )
+  (wire (pts (xy 228.6 52.07) (xy 250.19 52.07))
+    (stroke (width 0) (type default))
+  )
   (wire (pts (xy 116.84 147.32) (xy 125.73 147.32))
     (stroke (width 0) (type solid))
@@
   (wire (pts (xy 71.12 52.07) (xy 71.12 53.34))
     (stroke (width 0) (type solid))
-  )
-  (wire (pts (xy 228.6 52.07) (xy 241.3 52.07))
-    (stroke (width 0) (type default))
   )
   (wire (pts (xy 212.09 62.23) (xy 217.17 62.23))
@@
     (effects (font (size 2.0066 2.0066)) (justify left))
   )
-  (hierarchical_label "+3.3v" (shape input) (at 241.3 52.07 0) (fields_autoplaced)
+  (hierarchical_label "+3.3v" (shape input) (at 250.19 52.07 0) (fields_autoplaced)
     (effects (font (size 1.27 1.27)) (justify left))
   )

Commit message: - BOM added (Farnell nrs)
Parts:
- C13: value 100n 100v -> 100n; Farnell (none) -> 1414664
- C14, C15, C16, C17, C19, C20, C21, C27, C28, C29, C31: Farnell (none) -> 2611943
- C18, C22, C23: Farnell (none) -> 1414664
- C24, C26: value nf -> 220p; Farnell (none) -> 2896723
- C25: Farnell (none) -> 1759229
- C30: Farnell (none) -> 9406352
- C32: Farnell (none) -> 3013482
- C33: Farnell (none) -> 4144905
- D3: Farnell (none) -> 1431244
- J3: Farnell (none) -> 3041165
- L1: Farnell (none) -> 2616889
- Q1: Farnell (none) -> 3405192
- R18, R21: Farnell (none) -> 1469865
- R19: Farnell (none) -> 3235140
- R20: Farnell (none) -> 1469893
- R22: Farnell (none) -> 1576464
- U6: Farnell (none) -> 3518317
- U7: Farnell (none) -> 4027203
Changed lines of the file:
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@@
+      (effects (font (size 1.27 1.27)) hide)
+    )
+    (property "Farnell" "2611943" (at 203.2 115.57 0)
       (effects (font (size 1.27 1.27)) hide)
     )
@@
       (effects (font (size 1.27 1.27)) hide)
     )
+    (property "Farnell" "2611943" (at 193.04 115.57 0)
+      (effects (font (size 1.27 1.27)) hide)
+    )
     (pin "1")
     (pin "2")
@@
       (effects (font (size 1.27 1.27)) (justify left))
     )
-    (property "Value" "nf" (at 176.53 125.73 0)
+    (property "Value" "220p" (at 176.53 125.73 0)
       (effects (font (size 1.27 1.27)) (justify left))
     )
@@
       (effects (font (size 1.27 1.27)) hide)
     )
+    (property "Farnell" "2896723" (at 173.99 123.19 0)
+      (effects (font (size 1.27 1.27)) hide)
+    )
     (pin "1")
     (pin "2")
@@
       (effects (font (size 1.27 1.27)) hide)
     )
+    (property "Farnell" "1469865" (at 163.83 123.19 0)
+      (effects (font (size 1.27 1.27)) hide)
+    )
     (pin "1")
     (pin "2")
@@
       (effects (font (size 1.27 1.27)) hide)
     )
+    (property "Farnell" "2611943" (at 71.12 129.54 0)
+      (effects (font (size 1.27 1.27)) hide)
+    )
     (pin "1")
     (pin "2")
@@
     )
     (property "Field8" "" (at 59.69 129.54 0)
+      (effects (font (size 1.27 1.27)) hide)
+    )
+    (property "Farnell" "2611943" (at 59.69 129.54 0)
       (effects (font (size 1.27 1.27)) hide)
     )
@@
       (effects (font (size 1.27 1.27)) hide)
     )
+    (property "Farnell" "3041165" (at 34.29 45.72 0)
+      (effects (font (size 1.27 1.27)) hide)
+    )
     (pin "1")
     (pin "2")
@@
       (effects (font (size 1.27 1.27)) hide)
     )
+    (property "Farnell" "2611943" (at 81.28 129.54 0)
+      (effects (font (size 1.27 1.27)) hide)
+    )
     (pin "1")
     (pin "2")
@@
       (effects (font (size 1.27 1.27)) hide)
     )
+    (property "Farnell" "2611943" (at 110.49 46.99 0)
+      (effects (font (size 1.27 1.27)) hide)
+    )
     (pin "1")
     (pin "2")
@@
       (effects (font (size 1.27 1.27)) hide)
     )
+    (property "Farnell" "1431244" (at 71.12 48.26 0)
+      (effects (font (size 1.27 1.27)) hide)
+    )
     (pin "1")
     (pin "2")
@@
     )
     (property "Part Description" "Resistor 20K M1005 1% 63mW" (at 153.67 135.89 0)
+      (effects (font (size 1.27 1.27)) hide)
+    )
+    (property "Farnell" "1469893" (at 153.67 135.89 0)
       (effects (font (size 1.27 1.27)) hide)
     )
@@
       (effects (font (size 1.27 1.27)) (justify left))
     )
-    (property "Value" "nf" (at 146.05 142.24 0)
+    (property "Value" "220p" (at 146.05 142.24 0)
       (effects (font (size 1.27 1.27)) (justify left))
     )
@@
     )
     (property "Part Description" "" (at 143.51 139.7 0)
+      (effects (font (size 1.27 1.27)) hide)
+    )
+    (property "Farnell" "2896723" (at 143.51 139.7 0)
       (effects (font (size 1.27 1.27)) hide)
     )
@@
     )
     (property "Part Description" "DMP3013SFV-7 -  Power MOSFET, P Channel, 30 V, 12 A, 0.008 ohm, PowerDI3333, Surface Mount" (at 63.5 45.72 0)
+      (effects (font (size 1.27 1.27)) hide)
+    )
+    (property "Farnell" "3405192" (at 63.5 45.72 0)
       (effects (font (size 1.27 1.27)) hide)
     )
@@
       (effects (font (size 1.27 1.27)) hide)
     )
+    (property "Farnell" "1414664" (at 113.03 118.11 0)
+      (effects (font (size 1.27 1.27)) hide)
+    )
     (pin "1")
     (pin "2")
@@
     )
     (property "Field8" "120889581" (at 163.83 142.24 0)
+      (effects (font (size 1.27 1.27)) hide)
+    )
+    (property "Farnell" "1576464" (at 163.83 142.24 0)
       (effects (font (size 1.27 1.27)) hide)
     )
@@
       (effects (font (size 1.27 1.27)) hide)
     )
+    (property "Farnell" "2611943" (at 222.25 115.57 0)
+      (effects (font (size 1.27 1.27)) hide)
+    )
     (pin "1")
     (pin "2")
@@
       (effects (font (size 1.27 1.27)) (justify left))
     )
-    (property "Value" "100n 100v" (at 45.72 55.88 0)
+    (property "Value" "100n" (at 45.72 55.88 0)
       (effects (font (size 1.27 1.27)) (justify left))
     )
@@
       (effects (font (size 1.27 1.27)) hide)
     )
+    (property "Farnell" "1414664" (at 49.53 49.53 0)
+      (effects (font (size 1.27 1.27)) hide)
+    )
     (pin "1")
     (pin "2")
@@
     )
     (property "Field8" "" (at 102.87 129.54 0)
+      (effects (font (size 1.27 1.27)) hide)
+    )
+    (property "Farnell" "2611943" (at 102.87 129.54 0)
       (effects (font (size 1.27 1.27)) hide)
     )
@@
       (effects (font (size 1.27 1.27)) hide)
     )
+    (property "Farnell" "3013482" (at 228.6 58.42 0)
+      (effects (font (size 1.27 1.27)) hide)
+    )
     (pin "1")
     (pin "2")
@@
       (effects (font (size 1.27 1.27)) hide)
     )
+    (property "Farnell" "2611943" (at 49.53 129.54 0)
+      (effects (font (size 1.27 1.27)) hide)
+    )
     (pin "1")
     (pin "2")
@@
     )
     (property "Field8" "" (at 91.44 129.54 0)
+      (effects (font (size 1.27 1.27)) hide)
+    )
+    (property "Farnell" "2611943" (at 91.44 129.54 0)
       (effects (font (size 1.27 1.27)) hide)
     )
@@
       (effects (font (size 1.27 1.27)) hide)
     )
+    (property "Farnell" "3235140" (at 118.11 111.76 0)
+      (effects (font (size 1.27 1.27)) hide)
+    )
     (pin "1")
     (pin "2")
@@
       (effects (font (size 1.27 1.27)) hide)
     )
+    (property "Farnell" "1759229" (at 153.67 143.51 0)
+      (effects (font (size 1.27 1.27)) hide)
+    )
     (pin "1")
     (pin "2")
@@
       (effects (font (size 1.27 1.27)) hide)
     )
+    (property "Farnell" "1414664" (at 91.44 48.26 0)
+      (effects (font (size 1.27 1.27)) hide)
+    )
     (pin "1")
     (pin "2")
@@
       (effects (font (size 1.27 1.27)) hide)
     )
+    (property "Farnell" "1469865" (at 71.12 58.42 0)
+      (effects (font (size 1.27 1.27)) hide)
+    )
     (pin "1")
     (pin "2")
@@
       (effects (font (size 1.27 1.27)) hide)
     )
+    (property "Farnell" "2611943" (at 213.36 115.57 0)
+      (effects (font (size 1.27 1.27)) hide)
+    )
     (pin "1")
     (pin "2")
@@
     )
     (property "Part Description" "Buck Switching Regulator IC Positive Adjustable 0.8V 1 Output 5A 8-SOIC (0.154\", 3.90mm Width) Exposed Pad" (at 125.73 125.73 0)
+      (effects (font (size 1.27 1.27)) hide)
+    )
+    (property "Farnell" "3518317" (at 125.73 125.73 0)
       (effects (font (size 1.27 1.27)) hide)
     )
@@
       (effects (font (size 1.27 1.27)) hide)
     )
+    (property "Farnell" "2616889" (at 154.94 111.76 0)
+      (effects (font (size 1.27 1.27)) hide)
+    )
     (pin "1")
     (pin "2")
@@
     )
     (property "Part Description" "Capacitor, SP-Cap, 100u, 6.3V, 15mR ESR" (at 236.22 115.57 0)
+      (effects (font (size 1.27 1.27)) hide)
+    )
+    (property "Farnell" "4144905" (at 236.22 115.57 0)
       (effects (font (size 1.27 1.27)) hide)
     )
@@
       (effects (font (size 1.27 1.27)) hide)
     )
+    (property "Farnell" "4027203" (at 198.12 54.61 0)
+      (effects (font (size 1.27 1.27)) hide)
+    )
     (pin "1")
     (pin "5")
@@
       (effects (font (size 1.27 1.27)) hide)
     )
+    (property "Farnell" "9406352" (at 217.17 58.42 0)
+      (effects (font (size 1.27 1.27)) hide)
+    )
     (pin "1")
     (pin "2")
@@
       (effects (font (size 1.27 1.27)) hide)
     )
+    (property "Farnell" "1414664" (at 116.84 139.7 0)
+      (effects (font (size 1.27 1.27)) hide)
+    )
