File: pcb/USB_Sound.kicad_sch (KiCad schematic)
At the start: 37 parts, among them IC1 PCM2706, J2 USB4500-03-0-A_REVA, U4 FSUSB42MUX, U5 24AA02-OT, Y1 12Mhz

Commit message: - component selection/place
Parts:
- removed C2: 1u, Capacitor_SMD:CP_Elec_6.3x7.7, symbol Device:C_Polarized
- removed J2: USB4500-03-0-A_REVA, Footprints:GCT_USB4500-03-0-A_REVA, symbol USB4500-03-0-A_REVA:USB4500-03-0-A_REVA
- added C10, C11, C2: 1u, Capacitor_SMD:C_0805_2012Metric_Pad1.18x1.45mm_HandSolder, symbol Device:C
- added C12: 100n, Capacitor_SMD:C_0805_2012Metric_Pad1.18x1.45mm_HandSolder, symbol Device:C
- added J5: USB4085-GF-A_REVB, Footprints:GCT_USB4085-GF-A_REVB, symbol USB4085-GF-A_REVB:USB4085-GF-A_REVB
- C3, C8, C9: footprint Capacitor_SMD:CP_Elec_6.3x7.7 -> Capacitor_SMD:CP_Elec_6.3x3.9
- TP10: renamed from TP7; footprint TestPoint:TestPoint_Bridge_Pitch2.54mm_Drill1.0mm -> TestPoint:TestPoint_Bridge_Pitch2.0mm_Drill0.7mm
- TP11: renamed from TP8; footprint TestPoint:TestPoint_Bridge_Pitch2.54mm_Drill1.0mm -> TestPoint:TestPoint_THTPad_1.0x1.0mm_Drill0.5mm
- TP12: renamed from TP9; footprint TestPoint:TestPoint_Bridge_Pitch2.54mm_Drill1.0mm -> TestPoint:TestPoint_THTPad_1.0x1.0mm_Drill0.5mm
- TP7: renamed from TP4; footprint TestPoint:TestPoint_Bridge_Pitch2.54mm_Drill1.0mm -> TestPoint:TestPoint_THTPad_1.0x1.0mm_Drill0.5mm
- TP8: renamed from TP5; footprint TestPoint:TestPoint_Bridge_Pitch2.54mm_Drill1.0mm -> TestPoint:TestPoint_THTPad_1.0x1.0mm_Drill0.5mm
- TP9: renamed from TP6; footprint TestPoint:TestPoint_Bridge_Pitch2.54mm_Drill1.0mm -> TestPoint:TestPoint_Bridge_Pitch2.0mm_Drill0.7mm
- renumbered R9 to R10, R10 to R11, R11 to R12, R12 to R13, R13 to R14, R14 to R15, R15 to R16, R16 to R17, R6 to R7, R7 to R8, R8 to R9, TP10 to TP13, TP11 to TP14, TP3 to TP6
Connections:
- net +3.3v: now also C10.1, C11.1, C12.1, C2.2
- net GND: now also C10.2, C11.2, C12.2, C2.1, J5.A1 (GND), J5.A12 (GND), J5.B1 (GND), J5.B12 (GND), J5.S1 (SHELL), J5.S2 (SHELL), J5.S3 (SHELL), J5.S4 (SHELL)
- net USBD_N: now also J5.A7 (DN1), J5.B7 (DN2)
- net USBD_P: now also J5.A6 (DP1), J5.B6 (DP2)
- net at R9.1: now also J5.A4 (VBUS), J5.A9 (VBUS), J5.B4 (VBUS), J5.B9 (VBUS)

Commit message: - routed
Parts:
- renumbered J5 to J2, TP11 to TP10, TP12 to TP11, TP13 to TP12, TP14 to TP13, TP6 to TP5, TP7 to TP6, TP8 to TP7, TP9 to TP8, TP10 to TP9
Connections:
- net USBS_N: now reaches IC1.22 (D-), TP10.1, U4.4 (D_N)
- net USBS_P: now reaches IC1.23 (D+), TP11.1, U4.3 (D_P)
Changed lines of the file:
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@@
+    (effects (font (size 1.27 1.27)) (justify left bottom))
+  )
+  (label "USBS_P" (at 113.03 74.93 0) (fields_autoplaced)
     (effects (font (size 1.27 1.27)) (justify left bottom))
   )
@@
   )
   (label "I2S.LRCK" (at 50.8 133.35 0) (fields_autoplaced)
+    (effects (font (size 1.27 1.27)) (justify left bottom))
+  )
+  (label "USBS_N" (at 113.03 77.47 0) (fields_autoplaced)
     (effects (font (size 1.27 1.27)) (justify left bottom))
   )
@@
   (symbol (lib_id "Connector:TestPoint") (at 119.38 86.36 0) (unit 1)
     (in_bom yes) (on_board yes) (dnp no)
-    (property "Reference" "TP11" (at 114.3 85.09 0)
+    (property "Reference" "TP10" (at 114.3 85.09 0)
       (effects (font (size 1.27 1.27)) (justify left))
     )
@@
       (project "VolumioAmp"
         (path "/c639bae0-d26f-43ee-9e8c-ca060284bd0b/93301fd2-7a6d-48be-bd24-243a1877e343"
-          (reference "TP11") (unit 1)
+          (reference "TP10") (unit 1)
         )
       )
@@
   (symbol (lib_id "Connector:TestPoint") (at 46.99 128.27 90) (unit 1)
     (in_bom yes) (on_board yes) (dnp no)
-    (property "Reference" "TP6" (at 41.91 127 90)
+    (property "Reference" "TP5" (at 41.91 127 90)
       (effects (font (size 1.27 1.27)) (justify left))
     )
@@
       (project "VolumioAmp"
         (path "/c639bae0-d26f-43ee-9e8c-ca060284bd0b/93301fd2-7a6d-48be-bd24-243a1877e343"
-          (reference "TP6") (unit 1)
+          (reference "TP5") (unit 1)
         )
       )
@@
   (symbol (lib_id "USB4085-GF-A_REVB:USB4085-GF-A_REVB") (at 38.1 48.26 0) (mirror y) (unit 1)
     (in_bom yes) (on_board yes) (dnp no)
-    (property "Reference" "J5" (at 38.1 71.12 0)
+    (property "Reference" "J2" (at 38.1 71.12 0)
       (effects (font (size 1.27 1.27)))
     )
@@
       (project "VolumioAmp"
         (path "/c639bae0-d26f-43ee-9e8c-ca060284bd0b/93301fd2-7a6d-48be-bd24-243a1877e343"
-          (reference "J5") (unit 1)
+          (reference "J2") (unit 1)
         )
       )
@@
   (symbol (lib_id "Connector:TestPoint") (at 127 86.36 0) (unit 1)
     (in_bom yes) (on_board yes) (dnp no)
-    (property "Reference" "TP12" (at 129.54 85.09 0)
+    (property "Reference" "TP11" (at 129.54 85.09 0)
       (effects (font (size 1.27 1.27)) (justify left))
     )
@@
       (project "VolumioAmp"
         (path "/c639bae0-d26f-43ee-9e8c-ca060284bd0b/93301fd2-7a6d-48be-bd24-243a1877e343"
-          (reference "TP12") (unit 1)
+          (reference "TP11") (unit 1)
         )
       )
@@
   (symbol (lib_id "Connector:TestPoint") (at 196.85 97.79 270) (unit 1)
     (in_bom yes) (on_board yes) (dnp no)
-    (property "Reference" "TP13" (at 199.39 95.25 90)
+    (property "Reference" "TP12" (at 199.39 95.25 90)
       (effects (font (size 1.27 1.27)) (justify left))
     )
@@
       (project "VolumioAmp"
         (path "/c639bae0-d26f-43ee-9e8c-ca060284bd0b/93301fd2-7a6d-48be-bd24-243a1877e343"
-          (reference "TP13") (unit 1)
+          (reference "TP12") (unit 1)
         )
       )
@@
   (symbol (lib_id "Connector:TestPoint") (at 110.49 172.72 0) (unit 1)
     (in_bom yes) (on_board yes) (dnp no)
-    (property "Reference" "TP9" (at 113.03 173.99 0)
+    (property "Reference" "TP8" (at 113.03 173.99 0)
       (effects (font (size 1.27 1.27)) (justify left))
     )
@@
       (project "VolumioAmp"
         (path "/c639bae0-d26f-43ee-9e8c-ca060284bd0b/93301fd2-7a6d-48be-bd24-243a1877e343"
-          (reference "TP9") (unit 1)
+          (reference "TP8") (unit 1)
         )
       )
@@
   (symbol (lib_id "Connector:TestPoint") (at 68.58 86.36 180) (unit 1)
     (in_bom yes) (on_board yes) (dnp no)
-    (property "Reference" "TP8" (at 66.04 87.63 0)
+    (property "Reference" "TP7" (at 66.04 87.63 0)
       (effects (font (size 1.27 1.27)) (justify left))
     )
@@
       (project "VolumioAmp"
         (path "/c639bae0-d26f-43ee-9e8c-ca060284bd0b/93301fd2-7a6d-48be-bd24-243a1877e343"
-          (reference "TP8") (unit 1)
+          (reference "TP7") (unit 1)
         )
       )
@@
   (symbol (lib_id "Connector:TestPoint") (at 196.85 102.87 270) (unit 1)
     (in_bom yes) (on_board yes) (dnp no)
-    (property "Reference" "TP14" (at 199.39 100.33 90)
+    (property "Reference" "TP13" (at 199.39 100.33 90)
       (effects (font (size 1.27 1.27)) (justify left))
     )
@@
       (project "VolumioAmp"
         (path "/c639bae0-d26f-43ee-9e8c-ca060284bd0b/93301fd2-7a6d-48be-bd24-243a1877e343"
-          (reference "TP14") (unit 1)
+          (reference "TP13") (unit 1)
         )
       )
@@
   (symbol (lib_id "Connector:TestPoint") (at 68.58 78.74 0) (unit 1)
     (in_bom yes) (on_board yes) (dnp no)
-    (property "Reference" "TP7" (at 71.12 77.47 0)
+    (property "Reference" "TP6" (at 71.12 77.47 0)
       (effects (font (size 1.27 1.27)) (justify left))
     )
@@
       (project "VolumioAmp"
         (path "/c639bae0-d26f-43ee-9e8c-ca060284bd0b/93301fd2-7a6d-48be-bd24-243a1877e343"
-          (reference "TP7") (unit 1)
+          (reference "TP6") (unit 1)
         )
       )
@@
   (symbol (lib_id "Connector:TestPoint") (at 116.84 179.07 180) (unit 1)
     (in_bom yes) (on_board yes) (dnp no)
-    (property "Reference" "TP10" (at 114.3 180.34 0)
+    (property "Reference" "TP9" (at 114.3 180.34 0)
       (effects (font (size 1.27 1.27)) (justify left))
     )
@@
       (project "VolumioAmp"
         (path "/c639bae0-d26f-43ee-9e8c-ca060284bd0b/93301fd2-7a6d-48be-bd24-243a1877e343"
-          (reference "TP10") (unit 1)
-        )
-      )
+          (reference "TP9") (unit 1)
+        )
+      )

Commit message: - routed
Parts:
- added JP5: SDA, Jumper:SolderJumper-2_P1.3mm_Open_TrianglePad1.0x1.5mm, symbol Jumper:SolderJumper_2_Open
- added JP7: SCL, Jumper:SolderJumper-2_P1.3mm_Open_TrianglePad1.0x1.5mm, symbol Jumper:SolderJumper_2_Open
- renumbered JP5 to JP6, JP6 to JP8, JP7 to JP9
Connections:
- net SCL: now also JP7.1 (A); no longer IC1.14 (CK), R12.2, TP9.1, U5.1 (SCL)
- net SDA: now also JP5.1 (A); no longer IC1.15 (DT), R10.2, TP8.1, U5.3 (SDA)
- new net: IC1.14 (CK), JP7.2 (B), R12.2, TP9.1, U5.1 (SCL)
- new net: IC1.15 (DT), JP5.2 (B), R10.2, TP8.1, U5.3 (SDA)

Commit message: - BOM added (Farnell nrs)
Parts:
- C10, C11, C2: Farnell (none) -> 3013482
- C12: Farnell (none) -> 1414664
- C3: Farnell (none) -> 1834254
- C4, C5: value 22n -> 22p; Farnell (none) -> 2896721
- C6, C7: Farnell (none) -> 1828943
- C8, C9: Farnell (none) -> 1187011
- IC1: Farnell (none) -> 3118707
- J2: Farnell (none) -> 2924867
- R10, R12: Farnell (none) -> 3392813
- R11, R13: Farnell (none) -> 2138741
- R14, R15, R16, R17: Farnell (none) -> 2861528
- R7: Farnell (none) -> 3546693
- R8: Farnell (none) -> 3598538
- R9: Farnell (none) -> 1576464
- U4: Farnell (none) -> 2564479
- U5: Farnell (none) -> 3861413
Changed lines of the file:
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@@
+      (effects (font (size 1.27 1.27)) hide)
+    )
+    (property "Farnell" "2861528" (at 151.13 109.22 0)
       (effects (font (size 1.27 1.27)) hide)
     )
@@
       (effects (font (size 1.27 1.27)) hide)
     )
+    (property "Farnell" "1834254" (at 71.12 115.57 0)
+      (effects (font (size 1.27 1.27)) hide)
+    )
     (pin "1")
     (pin "2")
@@
       (effects (font (size 1.27 1.27)) hide)
     )
+    (property "Farnell" "1187011" (at 171.45 102.87 0)
+      (effects (font (size 1.27 1.27)) hide)
+    )
     (pin "1")
     (pin "2")
@@
       (effects (font (size 1.27 1.27)) hide)
     )
+    (property "Farnell" "3013482" (at 58.42 123.19 0)
+      (effects (font (size 1.27 1.27)) hide)
+    )
     (pin "1")
     (pin "2")
@@
     )
     (property "Datasheet" "~" (at 156.21 109.22 0)
+      (effects (font (size 1.27 1.27)) hide)
+    )
+    (property "Farnell" "2861528" (at 156.21 109.22 0)
       (effects (font (size 1.27 1.27)) hide)
     )
@@
       (effects (font (size 1.27 1.27)) hide)
     )
+    (property "Farnell" "2861528" (at 182.88 109.22 0)
+      (effects (font (size 1.27 1.27)) hide)
+    )
     (pin "1")
     (pin "2")
@@
     )
     (property "Datasheet" "~" (at 181.61 146.05 0)
+      (effects (font (size 1.27 1.27)) hide)
+    )
+    (property "Farnell" "3013482" (at 181.61 146.05 0)
       (effects (font (size 1.27 1.27)) hide)
     )
@@
       (effects (font (size 1.27 1.27)) (justify left))
     )
-    (property "Value" "22n" (at 107.95 187.96 0)
+    (property "Value" "22p" (at 107.95 187.96 0)
       (effects (font (size 1.27 1.27)) (justify left))
     )
@@
       (effects (font (size 1.27 1.27)) hide)
     )
+    (property "Farnell" "2896721" (at 104.14 186.69 0)
+      (effects (font (size 1.27 1.27)) hide)
+    )
     (pin "2")
     (pin "1")
@@
     )
     (property "Datasheet" "http://ww1.microchip.com/downloads/en/DeviceDoc/21709J.pdf" (at 151.13 177.8 0)
+      (effects (font (size 1.27 1.27)) hide)
+    )
+    (property "Farnell" "3861413" (at 151.13 177.8 0)
       (effects (font (size 1.27 1.27)) hide)
     )
@@
     (property "Check_prices" "https://www.snapeda.com/parts/PCM2706/Burr+Brown/view-part/?ref=eda" (at 99.06 130.81 0)
       (effects (font (size 1.27 1.27)) (justify bottom) hide)
+    )
+    (property "Farnell" "3118707" (at 99.06 130.81 0)
+      (effects (font (size 1.27 1.27)) hide)
     )
     (pin "1")
@@
       (effects (font (size 1.27 1.27)) hide)
     )
+    (property "Farnell" "2138741" (at 135.89 118.11 0)
+      (effects (font (size 1.27 1.27)) hide)
+    )
     (pin "1")
     (pin "2")
@@
       (effects (font (size 1.27 1.27)) hide)
     )
+    (property "Farnell" "3598538" (at 96.52 173.99 0)
+      (effects (font (size 1.27 1.27)) hide)
+    )
     (pin "1")
     (pin "2")
@@
       (effects (font (size 1.27 1.27)) hide)
     )
+    (property "Farnell" "3392813" (at 135.89 167.64 0)
+      (effects (font (size 1.27 1.27)) hide)
+    )
     (pin "2")
     (pin "1")
@@
       (effects (font (size 1.27 1.27)) hide)
     )
+    (property "Farnell" "1828943" (at 135.89 109.22 0)
+      (effects (font (size 1.27 1.27)) hide)
+    )
     (pin "1")
     (pin "2")
@@
       (effects (font (size 1.27 1.27)) (justify left))
     )
-    (property "Value" "22n" (at 82.55 187.96 0)
+    (property "Value" "22p" (at 82.55 187.96 0)
       (effects (font (size 1.27 1.27)) (justify left))
     )
@@
     )
     (property "Datasheet" "~" (at 87.63 186.69 0)
+      (effects (font (size 1.27 1.27)) hide)
+    )
+    (property "Farnell" "2896721" (at 87.63 186.69 0)
       (effects (font (size 1.27 1.27)) hide)
     )
@@
     (property "SNAPEDA_PN" "USB4085-GF-A" (at 38.1 48.26 0)
       (effects (font (size 1.27 1.27)) (justify bottom) hide)
+    )
+    (property "Farnell" "2924867" (at 38.1 48.26 0)
+      (effects (font (size 1.27 1.27)) hide)
     )
     (pin "A1")
@@
       (effects (font (size 1.27 1.27)) hide)
     )
+    (property "Farnell" "3013482" (at 172.72 146.05 0)
+      (effects (font (size 1.27 1.27)) hide)
+    )
     (pin "1")
     (pin "2")
@@
       (effects (font (size 1.27 1.27)) hide)
     )
+    (property "Farnell" "1828943" (at 142.24 109.22 0)
+      (effects (font (size 1.27 1.27)) hide)
+    )
     (pin "1")
     (pin "2")
@@
       (effects (font (size 1.27 1.27)) hide)
     )
+    (property "Farnell" "1187011" (at 161.29 100.33 0)
+      (effects (font (size 1.27 1.27)) hide)
+    )
     (pin "1")
     (pin "2")
@@
     )
     (property "Part Description" "USB Switch IC 1 Channel 10-MSOP" (at 91.44 85.09 0)
+      (effects (font (size 1.27 1.27)) hide)
+    )
+    (property "Farnell" "2564479" (at 91.44 85.09 0)
       (effects (font (size 1.27 1.27)) hide)
     )
@@
       (effects (font (size 1.27 1.27)) hide)
     )
+    (property "Farnell" "2138741" (at 142.24 118.11 0)
+      (effects (font (size 1.27 1.27)) hide)
+    )
     (pin "1")
     (pin "2")
@@
       (effects (font (size 1.27 1.27)) hide)
     )
+    (property "Farnell" "3392813" (at 132.08 167.64 0)
+      (effects (font (size 1.27 1.27)) hide)
+    )
     (pin "1")
     (pin "2")
@@
     )
     (property "Datasheet" "~" (at 176.53 109.22 0)
+      (effects (font (size 1.27 1.27)) hide)
+    )
+    (property "Farnell" "2861528" (at 176.53 109.22 0)
       (effects (font (size 1.27 1.27)) hide)
     )
@@
       (effects (font (size 1.27 1.27)) hide)
     )
+    (property "Farnell" "1576464" (at 105.41 46.99 0)
+      (effects (font (size 1.27 1.27)) hide)
+    )
     (pin "1")
     (pin "2")
@@
       (effects (font (size 1.27 1.27)) hide)
     )
+    (property "Farnell" "1414664" (at 189.23 146.05 0)
+      (effects (font (size 1.27 1.27)) hide)
+    )
     (pin "1")
     (pin "2")
@@
       (effects (font (size 1.27 1.27)) hide)
     )
+    (property "Farnell" "3546693" (at 46.99 123.19 0)
+      (effects (font (size 1.27 1.27)) hide)
+    )
