File: pcb/VolumioAmp.kicad_pcb (KiCad board)
At the start: 2 copper layers, 172.1 x 71.1 mm, 121 parts, among them IC1 PCM2706, IC2 WM8804GEDS_V, J1 L829-1J1T-43, J2 USB4500-03-0-A_REVA, J3 24v Input, J4 Screw_Terminal_01x04, J5 Conn_Coaxial, Q1 DMP3013SFV-7, U1 74LVC1G07SE-7, U2 TPD4EUSB30, U3 TPD4EUSB30, U4 FSUSB42MUX, U5 24AA02-OT, U6 AP64501SP-13, U7 LT1761-3.3, U8 MA12040PXUMA1, Y1 12Mhz, Y2 12Mhz

Commit message: - placing components
Parts:
- removed J5: Conn_Coaxial, Connector_Coaxial:BNC_PanelMountable_Vertical
- added R24: 470R, Resistor_SMD:R_0805_2012Metric_Pad1.20x1.40mm_HandSolder, B.Cu at (209.5, 59.3)
- added TP21: TestPoint, TestPoint:TestPoint_Bridge_Pitch2.54mm_Drill1.0mm, F.Cu at (133.5, 137.8)
- added TP22: TestPoint, TestPoint:TestPoint_Bridge_Pitch2.54mm_Drill1.0mm, F.Cu at (126.4, 138.0)
- C1, C10, R1, R4, R5, U2, U3: moved to B.Cu
- R8: value 2.2K 1% -> 2.2K
- moved C30 140.7 mm to (178.4, 115.4), turned to 90 degrees
- moved C35 137.1 mm to (61.5, 128.3)
- moved C28 136.6 mm to (183.5, 115.1), turned to 90 degrees
- moved C26 135.0 mm to (173.0, 118.0), turned to -90 degrees
- moved TP13 134.0 mm to (175.8, 58.6)
- moved R8 134.0 mm to (163.2, 126.2), turned to 90 degrees
- moved TP19 132.3 mm to (63.5, 116.0)
- moved TP16 131.6 mm to (62.2, 110.1)
- moved TP18 123.0 mm to (53.2, 110.6)
- moved C24 123.0 mm to (173.0, 112.9), turned to 90 degrees
- moved U4 114.2 mm to (169.4, 126.1)
- moved R4 112.1 mm to (210.0, 64.4), turned to 180 degrees
- moved C48 107.8 mm to (134.9, 134.2)
- moved TP14 107.5 mm to (176.3, 65.0)
- moved R20 107.3 mm to (148.1, 65.0), turned to -90 degrees
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Connections:
- J1 pad 17: unconnected-(J1-Pad17) -> Net-(J1-Pad17)
- Module1 pad 19: unconnected-(Module1A-Ethernet_nLED1(3.3v)-Pad19) -> Net-(Module1A-Ethernet_nLED1(3.3v))
Other:
- board size 172.1 x 71.1 mm -> 199.3 x 87 mm

Commit message: - component selection/place
Parts:
- removed J2: USB4500-03-0-A_REVA, Footprints:GCT_USB4500-03-0-A_REVA
- added C10: 1u, Capacitor_SMD:C_0805_2012Metric_Pad1.18x1.45mm_HandSolder, F.Cu at (120.8, 71.9)
- added C11: 1u, Capacitor_SMD:C_0805_2012Metric_Pad1.18x1.45mm_HandSolder, F.Cu at (125.7, 71.9)
- added C12: 100n, Capacitor_SMD:C_0805_2012Metric_Pad1.18x1.45mm_HandSolder, F.Cu at (133.6, 78.9)
- added J5: USB4085-GF-A_REVB, Footprints:GCT_USB4085-GF-A_REVB, F.Cu at (175.3, 58.0)
- added TP1: TestPoint, TestPoint:TestPoint_Bridge_Pitch2.54mm_Drill1.0mm, F.Cu at (200.7, 119.8)
- added TP3: TestPoint, TestPoint:TestPoint_Bridge_Pitch2.54mm_Drill1.0mm, F.Cu at (200.7, 127.9)
- C2: footprint Capacitor_SMD:CP_Elec_6.3x7.7 -> Capacitor_SMD:C_0805_2012Metric_Pad1.18x1.45mm_HandSolder
- C3, C8, C9: footprint Capacitor_SMD:CP_Elec_6.3x7.7 -> Capacitor_SMD:CP_Elec_6.3x3.9
- R9: renamed from R8; value 2.2K -> 2.2K 1%
- TP10: renamed from TP7; footprint TestPoint:TestPoint_Bridge_Pitch2.54mm_Drill1.0mm -> TestPoint:TestPoint_Bridge_Pitch2.0mm_Drill0.7mm
- TP11: renamed from TP8; footprint TestPoint:TestPoint_Bridge_Pitch2.54mm_Drill1.0mm -> TestPoint:TestPoint_THTPad_1.0x1.0mm_Drill0.5mm
- TP12: renamed from TP9; footprint TestPoint:TestPoint_Bridge_Pitch2.54mm_Drill1.0mm -> TestPoint:TestPoint_THTPad_1.0x1.0mm_Drill0.5mm
- TP16: renamed from TP13; footprint TestPoint:TestPoint_Bridge_Pitch2.54mm_Drill1.0mm -> TestPoint:TestPoint_Bridge_Pitch2.0mm_Drill0.7mm; moved to B.Cu
- TP17: renamed from TP14; footprint TestPoint:TestPoint_Bridge_Pitch2.54mm_Drill1.0mm -> TestPoint:TestPoint_Bridge_Pitch2.0mm_Drill0.7mm; moved to B.Cu
- TP24: renamed from TP21; footprint TestPoint:TestPoint_Bridge_Pitch2.54mm_Drill1.0mm -> TestPoint:TestPoint_Bridge_Pitch2.0mm_Drill0.7mm
- TP25: renamed from TP22; footprint TestPoint:TestPoint_Bridge_Pitch2.54mm_Drill1.0mm -> TestPoint:TestPoint_Bridge_Pitch2.0mm_Drill0.7mm
- TP4: renamed from TP1; footprint TestPoint:TestPoint_Bridge_Pitch2.54mm_Drill1.0mm -> TestPoint:TestPoint_THTPad_1.0x1.0mm_Drill0.5mm; moved to B.Cu
- TP7: renamed from TP4; footprint TestPoint:TestPoint_Bridge_Pitch2.54mm_Drill1.0mm -> TestPoint:TestPoint_THTPad_1.0x1.0mm_Drill0.5mm
- TP8: renamed from TP5; footprint TestPoint:TestPoint_Bridge_Pitch2.54mm_Drill1.0mm -> TestPoint:TestPoint_THTPad_1.0x1.0mm_Drill0.5mm
- TP9: renamed from TP6; footprint TestPoint:TestPoint_Bridge_Pitch2.54mm_Drill1.0mm -> TestPoint:TestPoint_Bridge_Pitch2.0mm_Drill0.7mm
- U2, U3: moved to F.Cu
- moved TP13 83.7 mm to (157.4, 58.8), turned to 90 degrees
- moved TP14 81.3 mm to (157.4, 66.2), turned to 90 degrees
- moved TP7 70.9 mm to (180.2, 71.6), turned to 90 degrees
- moved TP8 70.1 mm to (180.2, 69.5), turned to 90 degrees
- moved TP17 69.2 mm to (178.7, 134.2), turned to 90 degrees
- moved TP16 68.2 mm to (178.7, 126.7), turned to 90 degrees
- moved C14 66.3 mm to (143.3, 130.2)
- moved C19 66.3 mm to (139.4, 130.2)
- moved C15 66.3 mm to (139.4, 125.3)
- moved C16 66.3 mm to (143.3, 125.3)
- moved C17 66.3 mm to (135.6, 125.3)
- moved C22 66.3 mm to (147.7, 121.7)
- moved C24 66.3 mm to (152.8, 133.9)
- moved C26 66.3 mm to (163.9, 130.1)
- moved C28 66.3 mm to (167.4, 130.0)
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- renumbered C10 to C13, C11 to C14, C12 to C15, C13 to C16, C14 to C17, C15 to C18, C16 to C19, C17 to C20, C18 to C21, C19 to C22, C20 to C23, C21 to C24, C22 to C25, C23 to C26, C24 to C27, C25 to C28, C26 to C29, C27 to C30, C28 to C31, C29 to C32, C30 to C33, C31 to C34, C32 to C35, C33 to C36, C34 to C37, C35 to C38, C36 to C39, C37 to C40, C38 to C41, C39 to C42, C40 to C43, C41 to C44, C42 to C45, C43 to C46, C44 to C47, C45 to C48, C46 to C49, C47 to C50, C48 to C51, R9 to R10, R10 to R11, R11 to R12, R12 to R13, R13 to R14, R14 to R15, R15 to R16, R16 to R17, R17 to R18, R18 to R19, R19 to R20, R20 to R21, R21 to R22, R22 to R23, R23 to R24, R24 to R4, R4 to R5, R5 to R6, R6 to R7, R7 to R8, TP10 to TP13, TP11 to TP14, TP12 to TP15, TP15 to TP18, TP16 to TP19, TP17 to TP20, TP18 to TP21, TP19 to TP22, TP20 to TP23, TP3 to TP6
Connections:
- C2 pad 1: /I2STest/+3.3v -> GND
- C2 pad 2: GND -> /I2STest/+3.3v
- Module1 pad 92: unconnected-(Module1A-RUN_PG-Pad92) -> Net-(Module1A-RUN_PG)
- Module1 pad 93: unconnected-(Module1A-nRPIBOOT-Pad93) -> Net-(Module1A-nRPIBOOT)
- Module1 pad 99: unconnected-(Module1A-Global_EN-Pad99) -> Net-(Module1A-Global_EN)
- TP2 pad 1: Net-(D2-K) -> Net-(Module1A-nRPIBOOT)

Commit message: - wiring
Parts:
- TP1, TP2, TP3: footprint TestPoint:TestPoint_Bridge_Pitch2.54mm_Drill1.0mm -> TestPoint:TestPoint_THTPad_1.0x1.0mm_Drill0.5mm
- moved TP1 19.9 mm to (184.5, 131.4)
- moved TP3 16.3 mm to (184.4, 128.5)
- moved TP2 16.2 mm to (184.5, 125.1)
- moved C1 8.86 mm to (198.1, 81.5), turned to -90 degrees
- moved R6 2.97 mm to (194.1, 63.0), turned to -90 degrees
- moved TP8 2.80 mm to (180.1, 72.3)
- moved R9 2.80 mm to (171.4, 71.2)
- moved TP11 2.80 mm to (171.6, 77.6)
- moved TP12 2.80 mm to (171.6, 75.6)
- moved U4 2.80 mm to (175.8, 72.1)
- moved TP7 2.80 mm to (180.1, 74.4)
- moved D1 0.68 mm to (189.5, 70.6)
Routing:
- net /CM4_HighSpeed/USB2_P: track 0.00 -> 62.0 mm
- net /CM4_HighSpeed/USB2_N: track 0.00 -> 61.4 mm
- net /CM4_Ethernet/TRD0_P: track 0.00 -> 39.1 mm, vias 0 -> 2
- net /CM4_Ethernet/TRD0_N: track 0.00 -> 38.3 mm, vias 0 -> 2
- net /USB_Sound/USBD_N: track 0.00 -> 15.9 mm, vias 0 -> 2
- net /USB_Sound/USBD_P: track 0.00 -> 14.5 mm, vias 0 -> 2

Commit message: - component placed
Parts:
- TP16, TP17, TP4: moved to F.Cu
- moved TP21 70.9 mm to (101.9, 59.1), turned to 90 degrees
- moved TP22 59.6 mm to (81.5, 59.1), turned to 90 degrees
- moved TP19 58.9 mm to (91.7, 59.1), turned to 90 degrees
- moved TP18 58.5 mm to (86.6, 59.1), turned to 90 degrees
- moved TP20 55.8 mm to (96.8, 59.1), turned to 90 degrees
- moved C43 51.4 mm to (82.3, 106.3), turned to 90 degrees
- moved TP23 49.8 mm to (76.4, 59.1), turned to 90 degrees
- moved C39 49.4 mm to (88.4, 116.3)
- moved C45 43.9 mm to (88.4, 119.3)
- moved C48 42.2 mm to (82.8, 99.1)
- moved C2 39.7 mm to (114.8, 76.1), turned to -90 degrees
- moved C41 39.6 mm to (83.0, 124.3), turned to 90 degrees
- moved TP6 38.5 mm to (108.3, 82.3)
- moved C40 35.6 mm to (77.1, 124.3), turned to 90 degrees
- moved C36 35.5 mm to (70.0, 117.6)
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Connections:
- U8 pad 10: Net-(J4-Pin_2) -> Net-(J4-Pin_1)
- U8 pad 11: Net-(J4-Pin_2) -> Net-(J4-Pin_1)
- U8 pad 17: GND -> /CM4_Ethernet/+5v
- U8 pad 38: Net-(J4-Pin_4) -> Net-(J4-Pin_3)
- U8 pad 39: Net-(J4-Pin_4) -> Net-(J4-Pin_3)
- U8 pad 4: Net-(J4-Pin_1) -> Net-(J4-Pin_2)
- U8 pad 44: Net-(J4-Pin_3) -> Net-(J4-Pin_4)
- U8 pad 45: Net-(J4-Pin_3) -> Net-(J4-Pin_4)
- U8 pad 5: Net-(J4-Pin_1) -> Net-(J4-Pin_2)
Routing:
- net /Amplifier/+24v: track 0.00 -> 142.5 mm, vias 0 -> 2
- net /CM4_HighSpeed/USB2_P: track 62.0 -> 0.00 mm
- net /CM4_HighSpeed/USB2_N: track 61.4 -> 0.00 mm
- net /CM4_Ethernet/+5v: track 0.00 -> 56.2 mm
- net /CM4_Ethernet/TRD0_P: track 39.1 -> 0.00 mm, vias 2 -> 0
- net /CM4_Ethernet/TRD0_N: track 38.3 -> 0.00 mm, vias 2 -> 0
- net Net-(D3-A): track 0.00 -> 17.3 mm, vias 0 -> 2
- net /USB_Sound/USBD_N: track 15.9 -> 0.00 mm, vias 2 -> 0
- net /USB_Sound/USBD_P: track 14.5 -> 0.00 mm, vias 2 -> 0
- net Net-(J3-Pin_2): track 0.00 -> 10.1 mm
- net Net-(U6-SW): track 0.00 -> 8.32 mm
- net Net-(J4-Pin_4): track 0.00 -> 7.29 mm, vias 0 -> 2
Other:
- board size 199.3 x 87 mm -> 176 x 87 mm

Commit message: - routed
Parts:
- added C46: 1u, Capacitor_SMD:C_0805_2012Metric_Pad1.18x1.45mm_HandSolder, F.Cu at (96.2, 126.4)
- added C47: 1u, Capacitor_SMD:C_0805_2012Metric_Pad1.18x1.45mm_HandSolder, F.Cu at (101.3, 126.3)
- added C48: 1u, Capacitor_SMD:C_0805_2012Metric_Pad1.18x1.45mm_HandSolder, F.Cu at (86.1, 126.2)
- added C49: 1u, Capacitor_SMD:C_0805_2012Metric_Pad1.18x1.45mm_HandSolder, F.Cu at (91.1, 126.3)
- added L2: L, Inductor_SMD:L_0805_2012Metric, F.Cu at (97.1, 122.5)
- added L3: L, Inductor_SMD:L_0805_2012Metric, F.Cu at (102.3, 122.5)
- added L4: L, Inductor_SMD:L_0805_2012Metric, F.Cu at (87.1, 122.5)
- added L5: L, Inductor_SMD:L_0805_2012Metric, F.Cu at (92.1, 122.5)
- TP17: renamed from TP18; footprint TestPoint:TestPoint_Bridge_Pitch2.54mm_Drill1.0mm -> TestPoint:TestPoint_Bridge_Pitch2.0mm_Drill0.7mm
- TP18: renamed from TP19; footprint TestPoint:TestPoint_Bridge_Pitch2.54mm_Drill1.0mm -> TestPoint:TestPoint_Bridge_Pitch2.0mm_Drill0.7mm
- TP19: renamed from TP20; footprint TestPoint:TestPoint_Bridge_Pitch2.54mm_Drill1.0mm -> TestPoint:TestPoint_Bridge_Pitch2.0mm_Drill0.7mm
- TP20: renamed from TP21; footprint TestPoint:TestPoint_Bridge_Pitch2.54mm_Drill1.0mm -> TestPoint:TestPoint_Bridge_Pitch2.0mm_Drill0.7mm
- TP21: renamed from TP22; footprint TestPoint:TestPoint_Bridge_Pitch2.54mm_Drill1.0mm -> TestPoint:TestPoint_Bridge_Pitch2.0mm_Drill0.7mm
- TP22: renamed from TP23; footprint TestPoint:TestPoint_Bridge_Pitch2.54mm_Drill1.0mm -> TestPoint:TestPoint_Bridge_Pitch2.0mm_Drill0.7mm
- TP23: renamed from TP24; moved to B.Cu
- moved J3 92.2 mm to (134.9, 136.1), turned to 180 degrees
- moved TP23 92.1 mm to (79.1, 58.6), turned to 90 degrees
- moved TP24 91.4 mm to (73.4, 58.6), turned to 90 degrees
- moved C13 86.2 mm to (132.5, 132.9), turned to 0 degrees
- moved R18 79.7 mm to (123.9, 130.3), turned to 0 degrees
- moved C55 78.5 mm to (78.4, 68.3)
- moved R23 78.5 mm to (74.4, 65.7)
- moved R24 78.5 mm to (78.3, 64.8)
- moved Q1 76.4 mm to (129.8, 127.9), turned to -90 degrees
- moved D3 73.5 mm to (123.7, 125.8), turned to 90 degrees
- moved C18 68.9 mm to (129.7, 122.6), turned to 180 degrees
- moved TP14 66.3 mm to (123.6, 120.7), turned to 90 degrees
- moved IC2 64.4 mm to (79.0, 78.3), turned to 0 degrees
- moved C21 63.9 mm to (129.7, 119.1), turned to 180 degrees
- moved C30 59.0 mm to (104.0, 72.2)
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- renumbered C45 to C44, C44 to C45, C46 to C50, C47 to C51, C48 to C52, C49 to C53, C50 to C54, C51 to C55, J5 to J2, TP11 to TP10, TP12 to TP11, TP13 to TP12, TP14 to TP13, TP15 to TP14, TP16 to TP15, TP17 to TP16, TP25 to TP24, TP6 to TP5, TP7 to TP6, TP8 to TP7, TP9 to TP8, TP10 to TP9
Connections:
- net Net-(IC1-D+) renamed /USB_Sound/USBS_P
- net Net-(IC1-D-) renamed /USB_Sound/USBS_N
- U8 pad 10: Net-(J4-Pin_1) -> Net-(L3-Pad1)
- U8 pad 11: Net-(J4-Pin_1) -> Net-(L3-Pad1)
- U8 pad 38: Net-(J4-Pin_3) -> Net-(L5-Pad1)
- U8 pad 39: Net-(J4-Pin_3) -> Net-(L5-Pad1)
- U8 pad 4: Net-(J4-Pin_2) -> Net-(L2-Pad1)
- U8 pad 44: Net-(J4-Pin_4) -> Net-(L4-Pad1)
- U8 pad 45: Net-(J4-Pin_4) -> Net-(L4-Pad1)
- U8 pad 5: Net-(J4-Pin_2) -> Net-(L2-Pad1)
Routing:
- net GND: track 0.00 -> 207.2 mm, vias 0 -> 133
- net /Amplifier/SDA: track 0.00 -> 181.2 mm, vias 0 -> 5
- net /Amplifier/SCL: track 0.00 -> 180.2 mm, vias 0 -> 4
- net /Amplifier/I2S.BCK: track 0.00 -> 176.2 mm, vias 0 -> 6
- net /I2STest/+3.3v: track 0.00 -> 171.5 mm, vias 0 -> 3
- net /Amplifier/I2S.LRCK: track 0.00 -> 169.6 mm, vias 0 -> 3
- net /Amplifier/I2S.D: track 0.00 -> 164.4 mm, vias 0 -> 3
- net /CM4_Ethernet/+5v: track 56.2 -> 209.1 mm, vias 0 -> 4
- net /Amplifier/I2S.MCK: track 0.00 -> 118.4 mm, vias 0 -> 3
- net /Amplifier/AC.~{CLIP}: track 0.00 -> 113.5 mm, vias 0 -> 4
- net /Amplifier/AC.~{MUTE}: track 0.00 -> 109.5 mm, vias 0 -> 4
- net /Amplifier/AC.~{ENABLE}: track 0.00 -> 103.3 mm, vias 0 -> 4
- net /Amplifier/AC.~{ERROR}: track 0.00 -> 94.8 mm, vias 0 -> 2
- net /CM4_Ethernet/+3.3v: track 0.00 -> 65.1 mm
- net /CM4_HighSpeed/USB2_N: track 0.00 -> 63.1 mm, vias 0 -> 2
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- added copper zone on B.Cu, net GND
- added copper zone on F.Cu, net GND
- added copper zone on In1.Cu, net GND
- added copper zone on In2.Cu, net GND
Other:
- board size 176 x 87 mm -> 164.6 x 87 mm
- copper layers 2 -> 4
- rule solder_mask_min_width: 0.12 -> 0.1016

Commit message: - routed
Parts:
- added JP5: SDA, Jumper:SolderJumper-2_P1.3mm_Open_TrianglePad1.0x1.5mm, F.Cu at (134.1, 97.5)
- added JP7: SCL, Jumper:SolderJumper-2_P1.3mm_Open_TrianglePad1.0x1.5mm, F.Cu at (140.6, 97.5)
- TP23: moved to F.Cu
- moved TP9 5.98 mm to (141.6, 93.2), turned to 180 degrees
- moved TP8 5.65 mm to (135.2, 93.2), turned to 180 degrees
- moved R10 4.64 mm to (133.0, 88.0)
- moved R12 4.64 mm to (141.7, 88.0)
- moved U5 4.64 mm to (137.4, 88.0)
- moved C7 3.29 mm to (124.5, 61.7), turned to 180 degrees
- moved R14 1.29 mm to (134.4, 64.8), turned to 90 degrees
- moved C9 1.27 mm to (144.2, 65.5)
- moved C6 1.27 mm to (131.8, 68.1), turned to 180 degrees
- moved TP12 1.20 mm to (157.7, 59.9)
- moved R11 1.01 mm to (128.5, 64.8)
- moved TP13 0.74 mm to (157.7, 66.8)
- moved R17 0.68 mm to (152.1, 58.7)
- moved R15 0.64 mm to (127.6, 58.4)
- moved R2 0.50 mm to (189.5, 67.2)
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- renumbered JP5 to JP6, JP6 to JP8, JP7 to JP9
Connections:
- IC1 pad 14: /Amplifier/SCL -> Net-(IC1-CK)
- IC1 pad 15: /Amplifier/SDA -> Net-(IC1-DT)
- R10 pad 2: /Amplifier/SDA -> Net-(IC1-DT)
- R12 pad 2: /Amplifier/SCL -> Net-(IC1-CK)
- TP8 pad 1: /Amplifier/SDA -> Net-(IC1-DT)
- TP9 pad 1: /Amplifier/SCL -> Net-(IC1-CK)
- U5 pad 1: /Amplifier/SCL -> Net-(IC1-CK)
- U5 pad 3: /Amplifier/SDA -> Net-(IC1-DT)
Routing:
- net Net-(IC1-CK): track 0.00 -> 33.4 mm, vias 0 -> 1
- net /CM4_Ethernet/+5v: track 209.1 -> 236.6 mm, vias 4 -> 6
- net Net-(IC1-DT): track 0.00 -> 26.5 mm, vias 0 -> 1
- net /Amplifier/SDA: track 181.2 -> 155.3 mm, vias 5 -> 6
- net /Amplifier/SCL: track 180.2 -> 165.5 mm, vias 4 -> 5
- net /USB_Sound/USBD_P: track 27.9 -> 16.1 mm, vias 0 -> 2
- net /Amplifier/I2S.LRCK: track 169.6 -> 179.4 mm
- net /I2STest/+3.3v: track 171.5 -> 162.9 mm, vias 3 -> 2
- net /Amplifier/I2S.D: track 164.4 -> 172.3 mm
- net /Amplifier/AC.~{CLIP}: track 113.5 -> 106.4 mm, vias 4 -> 2
- net GND: track 207.2 -> 200.6 mm, vias 133 -> 170
- net Net-(IC1-VOUTL): track 23.4 -> 29.1 mm
- net /Amplifier/I2S.BCK: track 176.2 -> 180.9 mm, vias 6 -> 4
- net /Amplifier/AC.~{ENABLE}: track 103.3 -> 98.7 mm, vias 4 -> 2
- net /Amplifier/+24v: track 167.7 -> 171.9 mm
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
Commit message: - add production gerber
Other:
- board text added: "VolumioAmp-v0.1 (05/12/2023)"
Changed lines of the file:
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@@
   (gr_rect locked (start 66.9184 53.4365) (end 231.485 140.4315)
     (stroke (width 0.1) (type default)) (fill none) (layer "Edge.Cuts"))
+  (gr_text "VolumioAmp-v0.1 (05/12/2023)" (at 143.4592 138.0236) (layer "F.Cu")
+    (effects (font (size 1.524 1.524) (thickness 0.3048) bold) (justify left bottom))
+  )
   (segment (start 83.6879 87.9907) (end 82.8294 88.8492) (width 0.1524) (layer "F.Cu") (net 3))
   (segment (start 187.748 110.479) (end 187.1693 110.479) (width 0.1524) (layer "F.Cu") (net 3))

Commit message: - BOM added (Farnell nrs)
Parts:
- L2, L3, L4, L5: footprint Inductor_SMD:L_0805_2012Metric -> Inductor_SMD:L_Bourns_SRN6045TA
- moved L4 4.15 mm to (83.1, 123.5)
- moved C48 4.12 mm to (82.8, 128.8)
- moved C47 4.04 mm to (104.5, 128.8)
- moved L3 3.73 mm to (105.9, 123.5)
- moved C46 2.97 mm to (97.9, 128.8)
- moved C49 2.48 mm to (90.8, 128.8)
- moved L5 1.73 mm to (90.7, 123.5)
- moved L2 1.57 mm to (98.3, 123.5)
Routing:
- net GND: track 200.6 -> 194.9 mm, vias 170 -> 166
- net Net-(L4-Pad1): track 27.4 -> 30.0 mm
- net Net-(L3-Pad1): track 20.1 -> 22.5 mm
- net Net-(J4-Pin_1): track 13.6 -> 12.1 mm
- net Net-(J4-Pin_3): track 12.6 -> 11.3 mm
- net Net-(L5-Pad1): track 30.2 -> 29.0 mm
- net Net-(J4-Pin_2): track 12.6 -> 11.8 mm
- net Net-(L2-Pad1): track 19.0 -> 19.7 mm
Other:
- board text added: "VolumioAmp-v0.1 (06/12/2023)"
- board text removed: "VolumioAmp-v0.1 (05/12/2023)"
