File: testpcb/MA12040PTest/MA12040PTest.kicad_sch (KiCad schematic)
At the start: 94 parts, among them IC1 PCM2706, J2 USB4085-GF-A_REVB, J4 Screw_Terminal_01x04, U1 74LVC1G07SE-7, U4 FSUSB42MUX, U5 24AA02-OT, U6 AP64501SP-13, U7 LT1761-3.3, U8 MA12040PXUMA1, Y1 12Mhz

Commit message: - usb dac added
Parts:
- removed C10, C11, C2: 1u, Capacitor_SMD:C_0805_2012Metric_Pad1.18x1.45mm_HandSolder, symbol Device:C
- removed C12: 100n, Capacitor_SMD:C_0805_2012Metric_Pad1.18x1.45mm_HandSolder, symbol Device:C
- removed C3: 10u, Capacitor_SMD:CP_Elec_6.3x3.9, symbol Device:C_Polarized
- removed C4, C5: 22p, Capacitor_SMD:C_0805_2012Metric_Pad1.18x1.45mm_HandSolder, symbol Device:C
- removed C6, C7: 22n, Capacitor_SMD:C_0805_2012Metric_Pad1.18x1.45mm_HandSolder, symbol Device:C
- removed C8, C9: 100u, Capacitor_SMD:CP_Elec_6.3x3.9, symbol Device:C_Polarized
- removed IC1: PCM2706, Footprints:TQFP32-08, symbol PCM2706:PCM2706
- removed JP4: LRCK, Jumper:SolderJumper-2_P1.3mm_Open_TrianglePad1.0x1.5mm, symbol Jumper:SolderJumper_2_Open
- removed JP6: BCK, Jumper:SolderJumper-2_P1.3mm_Open_TrianglePad1.0x1.5mm, symbol Jumper:SolderJumper_2_Open
- removed JP7 (x4): SCL, Jumper:SolderJumper-2_P1.3mm_Open_TrianglePad1.0x1.5mm, symbol Jumper:SolderJumper_2_Open
- removed JP8: MCK, Jumper:SolderJumper-2_P1.3mm_Open_TrianglePad1.0x1.5mm, symbol Jumper:SolderJumper_2_Open
- removed JP9: D, Jumper:SolderJumper-2_P1.3mm_Open_TrianglePad1.0x1.5mm, symbol Jumper:SolderJumper_2_Open
- removed R10 (x2), R12 (x2): 1k5, Resistor_SMD:R_0805_2012Metric_Pad1.20x1.40mm_HandSolder, symbol Device:R
- removed R11, R13: 13R, Resistor_SMD:R_0805_2012Metric_Pad1.20x1.40mm_HandSolder, symbol Device:R
- removed R14, R15, R16, R17 (x3): 3k3, Resistor_SMD:R_0805_2012Metric_Pad1.20x1.40mm_HandSolder, symbol Device:R
- removed R7: 1k, Resistor_SMD:R_0805_2012Metric_Pad1.20x1.40mm_HandSolder, symbol Device:R
- removed R8: 1M, Resistor_SMD:R_0805_2012Metric_Pad1.20x1.40mm_HandSolder, symbol Device:R
- removed TP16, TP8, TP9: TestPoint, TestPoint:TestPoint_Bridge_Pitch2.0mm_Drill0.7mm, symbol Connector:TestPoint
- removed U5: 24AA02-OT, Package_TO_SOT_SMD:SOT-23-5, symbol Memory_EEPROM:24AA02-OT
- removed Y1: 12Mhz, Crystal:Crystal_SMD_Abracon_ABM3-2Pin_5.0x3.2mm_HandSoldering, symbol Device:Crystal
- added C13, C18, C32 (x4): 100n, Capacitor_SMD:C_0805_2012Metric_Pad1.18x1.45mm_HandSolder, symbol Device:C
- added C21: 10u 35v, Capacitor_SMD:C_0805_2012Metric_Pad1.18x1.45mm_HandSolder, symbol Device:C
- added C30: 10n, Capacitor_SMD:C_0805_2012Metric_Pad1.18x1.45mm_HandSolder, symbol Device:C
- added C32 (x2): 2n2, Capacitor_SMD:C_0805_2012Metric_Pad1.18x1.45mm_HandSolder, symbol Device:C
- added C32: 1u, Capacitor_SMD:C_0805_2012Metric_Pad1.18x1.45mm_HandSolder, symbol Device:C
- added C32 (x2): 2u2, Capacitor_SMD:C_0805_2012Metric_Pad1.18x1.45mm_HandSolder, symbol Device:C
- added C8 (x4): 10u, Capacitor_SMD:CP_Elec_6.3x3.9, symbol Device:C_Polarized
- added D2: SP0503BAHT, Package_TO_SOT_SMD:SOT-143, symbol Power_Protection:SP0503BAHT
- added D3: MMBZ5242BLT3G, Package_TO_SOT_SMD:SOT-23, symbol Diode:BZX84Cxx
- added J3: 24v Input, TerminalBlock:TerminalBlock_bornier-2_P5.08mm, symbol Connector:Screw_Terminal_01x02
- added JP5: FMT, Jumper:SolderJumper-3_P2.0mm_Open_TrianglePad1.0x1.5mm, symbol Jumper:SolderJumper_3_Open
- added JP7: LRCLK, Jumper:SolderJumper-2_P1.3mm_Open_TrianglePad1.0x1.5mm, symbol Jumper:SolderJumper_2_Open
- added JP7: MCLK, Jumper:SolderJumper-2_P1.3mm_Open_TrianglePad1.0x1.5mm, symbol Jumper:SolderJumper_2_Open
- added JP7: SCLK, Jumper:SolderJumper-2_P1.3mm_Open_TrianglePad1.0x1.5mm, symbol Jumper:SolderJumper_2_Open
- added JP7: D, Jumper:SolderJumper-2_P1.3mm_Open_TrianglePad1.0x1.5mm, symbol Jumper:SolderJumper_2_Open
- added Q1: DMP3013SFV-7, Package_SON:Diodes_PowerDI3333-8, symbol Transistor_FET:DMP3013SFV
- added R18: 12K 1%, Resistor_SMD:R_0805_2012Metric_Pad1.20x1.40mm_HandSolder, symbol Device:R
- added R22 (x4): 33R, Resistor_SMD:R_0805_2012Metric_Pad1.20x1.40mm_HandSolder, symbol Device:R
- added R22 (x4): 470R, Resistor_SMD:R_0805_2012Metric_Pad1.20x1.40mm_HandSolder, symbol Device:R
- added R22: 24k, Resistor_SMD:R_0805_2012Metric_Pad1.20x1.40mm_HandSolder, symbol Device:R
- added R22 (x2): 4k7, Resistor_SMD:R_0805_2012Metric_Pad1.20x1.40mm_HandSolder, symbol Device:R
- added R22 (x2): 1k5, Resistor_SMD:R_0805_2012Metric_Pad1.20x1.40mm_HandSolder, symbol Device:R
- added R22: 47k, Resistor_SMD:R_0805_2012Metric_Pad1.20x1.40mm_HandSolder, symbol Device:R
- added TP11 (x2): TestPoint, TestPoint:TestPoint_THTPad_1.0x1.0mm_Drill0.5mm, symbol Connector:TestPoint
- added TP14: TestPoint, TestPoint:TestPoint_Bridge_Pitch2.54mm_Drill1.0mm, symbol Connector:TestPoint
- added TP8 (x4): SCL, TestPoint:TestPoint_Bridge_Pitch2.0mm_Drill0.7mm, symbol Connector:TestPoint
- added TP9: L-Out, TestPoint:TestPoint_Bridge_Pitch2.0mm_Drill0.7mm, symbol Connector:TestPoint
- added TP9: R-Out, TestPoint:TestPoint_Bridge_Pitch2.0mm_Drill0.7mm, symbol Connector:TestPoint
- added TP9 (x2): TestPoint, TestPoint:TestPoint_Bridge_Pitch2.0mm_Drill0.7mm, symbol Connector:TestPoint
- added U10: PCM5101A, Package_SO:TSSOP-20_4.4x6.5mm_P0.65mm, symbol Audio:PCM5101A
- added U11: CP2615-xx-xM, Package_DFN_QFN:QFN-32-1EP_5x5mm_P0.5mm_EP3.3x3.3mm, symbol Interface_USB:CP2615-xx-xM
- added U7: LT1761-3.3, Package_TO_SOT_SMD:TSOT-23-5, symbol Regulator_Linear:LT1761-3.3
- JP11: value SDA -> MUTE; footprint (none) -> Jumper:SolderJumper-3_P2.0mm_Open_TrianglePad1.0x1.5mm
- JP12: value SCL -> ENABLE; footprint (none) -> Jumper:SolderJumper-3_P2.0mm_Open_TrianglePad1.0x1.5mm
- TP6: value TestPoint -> USB_P
- TP7: value TestPoint -> USB_N
Connections:
- net +24v is gone; now on net +12v: U8.41 (PVDD), U8.42 (PVDD), U8.7 (PVDD), U8.8 (PVDD)
- net AC.~{ENABLE} is gone; now on an unnamed net: U8.33 (~{ENABLE})
- net AC.~{MUTE} is gone; now on an unnamed net: U8.34 (~{MUTE})
- net I2S.BCK is gone; now on net BCK: U8.21 (SCK)
- net I2S.D is gone; now on net D: U8.23 (SD0)
- net I2S.LRCK is gone; now on net LRCK: U8.22 (WS)
- net I2S.MCK is gone; now on net MCK: U8.32 (CLK)
- net +3.3v: now also U1.5 (VCC), U1.5 (VCC), U1.5 (VCC), U1.5 (VCC), C32.1, C8.1, JP5.1 (A), R22.1, R22.1, R22.1, R22.1, R22.1, R22.2, U10.20 (DVDD), U11.6 (VDD), U11.7 (REGIN)
- net +5v: now also C26.1, C27.1, JP11.3 (B), JP12.3 (B), L1.2, R21.1, TP15.1, U8.51 (MSEL0), U7.1 (VIN), U7.3 (~{SHDN})
- net GND: now also C20.2, JP11.1 (A), JP12.1 (A), U1.3 (GND), U1.3 (GND), U1.3 (GND), U1.3 (GND), C13.2, C21.2, C32.2, C32.2, C32.2, C32.2, C32.2, C32.2, C32.2, C32.2, C8.2, C8.2, C8.2, C8.2, D2.1 (A), J3.1 (Pin_1), JP5.3 (B), R18.2, R22.1, R22.2, U10.10 (DEMP), U10.11 (FLT), U10.19 (DGND), U10.3 (CPGND), U10.9 (AGND), U11.3 (GND), U11.33 (GND), U7.2 (GND)
- net USBS_N: now also U11.5 (D-)
- net USBS_P: now also U11.4 (D+)
- net at C27.2, L2.2: now also J4.2 (Pin_2)
- net LRCK: now reaches U1.2
- net LRCK: now also U1.4, JP7.1 (A), R22.1, R22.2, TP8.1, U10.15 (LRCK)
- net +12v: now reaches C20.1, U6.2 (VIN), U6.3 (EN)
- net +12v: now also C18.1, C21.1, D3.3 (K), Q1.1 (S), Q1.2 (S), Q1.3 (S), TP14.1
- net at TP8.1, U8.30 (SDA): now also R22.2, U11.30 (I2C_SDA); no longer JP11.1 (A)
- net at TP8.1, U8.27 (SCL): now also R22.2, U11.29 (I2C_SCL); no longer JP12.1 (A)
- net at J2.A6 (DP1), J2.B6 (DP2), TP6.1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: now also D2.3 (K)
- net at J2.A4 (VBUS), J2.A9 (VBUS), J2.B4 (VBUS)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: now also D2.4 (K), TP9.1
- net at J2.A7 (DN1), J2.B7 (DN2), TP7.1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: now also D2.2 (K)
- net MCK: now reaches U1.2
- net MCK: now also U1.4, JP7.1 (A), R22.1, R22.2, TP8.1, U10.12 (SCK)
- net D: now reaches U1.2
- net D: now also U1.4, JP7.1 (A), R22.1, R22.2, TP8.1, U10.14 (DIN)
- net BCK: now reaches U1.2
- net BCK: now also U1.4, JP7.1 (A), R22.1, R22.2, TP8.1, U10.13 (BCK)
- net AC.~{CLIP}: no longer names the net of U8.15 (~{CLIP})
- net AC.~{ERROR}: no longer names the net of U8.16 (~{ERROR})
- new net: JP5.2 (C), U10.16 (FMT)
- new net: C18.2, D3.1 (A), Q1.4 (G), R18.1
- new net: C32.1, R22.1, TP9.1 (x2)
- new net: JP7.2 (B), U11.28 (I2S_LRCLK)
- new net: C30.1, C32.1, C32.1, C32.1, C8.1, C8.1, U10.1 (CPVDD), U10.8 (AVDD), U7.5 (VOUT)
- new net: R22.1, R22.2, TP9.1, U10.17 (XSMT)
- new net: R22.1, R22.2, TP11.1, U11.8 (VBUS)
- new net: R22.2, U11.9 (~{RST})
- new net: C30.2, U7.4 (BYP)
- new net: C13.1, J3.2 (Pin_2), Q1.5 (D)
- new net: C32.1, U10.5 (VNEG)
- new net: R22.2, U10.7 (OUTR)
- new net: C32.1, C8.1, U10.18 (LDOO)
- new net: C32.1, U10.2 (CAPP)
- new net: C32.2, U10.4 (CAPM)
- new net: R22.2, U10.6 (OUTL)
- new net: JP7.2 (B), U11.26 (I2S_MCLK)
- new net: R22.2, TP11.1, U11.21 (~{CFGMODE})
- new net: JP7.2 (B), U11.2 (I2S_SCLK)
- new net: JP7.2 (B), U11.32 (I2S_SDOUT)
- no-connect marks 9 -> 23
Other:
- note added: "Ideal diode to prevent reverse polarity at the input"
- moved on the sheet: C20, C22, C23, C24, C25, C26, C27, C30, C32, J2, J4, L1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

Commit message: - work in progress
Parts:
- removed C30: 10n, Capacitor_SMD:C_0805_2012Metric_Pad1.18x1.45mm_HandSolder, symbol Device:C
- removed U7: LT1761-3.3, Package_TO_SOT_SMD:TSOT-23-5, symbol Regulator_Linear:LT1761-3.3
- added C32 (x2), C4: 1u, Capacitor_SMD:C_0805_2012Metric_Pad1.18x1.45mm_HandSolder, symbol Device:C
- added C4 (x7): 100n, Capacitor_SMD:C_0805_2012Metric_Pad1.18x1.45mm_HandSolder, symbol Device:C
- added C4, C5: 22p, Capacitor_SMD:C_0805_2012Metric_Pad1.18x1.45mm_HandSolder, symbol Device:C
- added J3: Conn_02x03_Top_Bottom, Connector_PinHeader_2.54mm:PinHeader_2x03_P2.54mm_Vertical, symbol Connector_Generic:Conn_02x03_Top_Bottom
- added JP7 (x6): ~, Jumper:SolderJumper-2_P1.3mm_Open_TrianglePad1.0x1.5mm, symbol Jumper:SolderJumper_2_Open
- added JP7: USB-VBUS, Jumper:SolderJumper-2_P1.3mm_Bridged_Pad1.0x1.5mm, symbol Jumper:SolderJumper_2_Open
- added JP7: SolderJumper_2_Open, symbol Jumper:SolderJumper_2_Open
- added R22 (x13): 1k5, Resistor_SMD:R_0805_2012Metric_Pad1.20x1.40mm_HandSolder, symbol Device:R
- added R22: 1k, Resistor_SMD:R_0805_2012Metric_Pad1.20x1.40mm_HandSolder, symbol Device:R
- added R22 (x2): 10k, Resistor_SMD:R_0805_2012Metric_Pad1.20x1.40mm_HandSolder, symbol Device:R
- added TP8: RP_SDA, TestPoint:TestPoint_Bridge_Pitch2.0mm_Drill0.7mm, symbol Connector:TestPoint
- added TP8: RP_SCL, TestPoint:TestPoint_Bridge_Pitch2.0mm_Drill0.7mm, symbol Connector:TestPoint
- added TP9: Reset, TestPoint:TestPoint_Bridge_Pitch2.0mm_Drill0.7mm, symbol Connector:TestPoint
- added U12, U6: AP2112K-3.3, Package_TO_SOT_SMD:SOT-23-5, symbol Regulator_Linear:AP2112K-3.3
- added U13: RP2040, Package_DFN_QFN:QFN-56-1EP_7x7mm_P0.4mm_EP3.2x3.2mm, symbol MCU_RaspberryPi:RP2040
- added U7: S25FL064LABMFI010, Footprints:SOIC8_208MIL_CYP, symbol S25FL064LABMFI010:S25FL064LABMFI010
- added Y1: 12Mhz, Crystal:Crystal_SMD_Abracon_ABM3-2Pin_5.0x3.2mm_HandSoldering, symbol Device:Crystal
- C8: footprint Capacitor_SMD:CP_Elec_6.3x3.9 -> Capacitor_SMD:CP_Elec_5x5.8; Farnell 1187011 -> 3386122
- TP9: footprint TestPoint:TestPoint_Bridge_Pitch2.0mm_Drill0.7mm -> TestPoint:TestPoint_THTPad_1.0x1.0mm_Drill0.5mm
- renumbered JP11 to JP8, JP12 to JP9, U11 to U4, U10 to U5
Connections:
- net +3.3v: now also C4.1, C4.1, C4.1, C4.1, C4.1, C4.1, JP7.2 (B), R22.1, R22.1, R22.1, R22.1, R22.1, R22.1, R22.2, R22.2, U6.5 (VOUT), U7.8 (VCC)
- net +5v: now also C32.1, U12.1 (VIN), U12.3 (EN), U6.1 (VIN), U6.3 (EN)
- net GND: now also C32.2, C32.2, C4.1, C4.1, C4.2, C4.2, C4.2, C4.2, C4.2, C4.2, C4.2, C5.2, J3.1 (Pin_1), R22.2, R22.2, R22.2, R22.2, R22.2, R22.2, U12.2 (GND), U13.57 (GND), U6.2 (GND), U7.4 (VSS)
- net SOUND_RESET: now reaches R22.2, U4.9 (~{RST})
- net SOUND_RESET: now also JP7.1 (A), R22.1, R22.2
- net PICO_SCL: now reaches R22.2, TP8.1, U4.29 (I2C_SCL), U8.27 (SCL)
- net PICO_SCL: now also JP7.1 (A), R22.1, R22.2
- net PICO_SDA: now reaches R22.2, TP8.1, U4.30 (I2C_SDA), U8.30 (SDA)
- net PICO_SDA: now also JP7.1 (A), R22.1, R22.2
- net at D2.4 (K), J2.A4 (VBUS), J2.A9 (VBUS)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: now also R22.1; no longer TP9.1, U4.2 (SEL)
- net CFGMODE: now reaches R22.2, TP11.1, U4.21 (~{CFGMODE})
- net CFGMODE: now also JP7.1 (A), R22.1, R22.2
- new net: C4.2, C4.2, U13.23 (DVDD), U13.45 (VREG_VOUT), U13.50 (DVDD)
- new net: C32.1, U12.5 (VOUT), U13.1 (IOVDD), U13.10 (IOVDD), U13.22 (IOVDD), U13.33 (IOVDD), U13.42 (IOVDD), U13.43 (ADC_AVDD), U13.44 (VREG_IN), U13.48 (USB_VDD), U13.49 (IOVDD)
- new net: J3.2 (Pin_2), U13.24 (SWCLK)
- new net: J3.5 (Pin_5), JP7.1 (A)
- new net: J3.6 (Pin_6), U13.25 (SWD)
- new net: R22.1, U13.21 (XOUT)
- new net: C5.1, R22.2, Y1.2
- new net: JP7.2 (B), U13.15 (GPIO12)
- new net: C4.1, U13.20 (XIN), Y1.1
- new net: JP7.2 (B), U13.13 (GPIO10)
- new net: JP7.2 (B), U13.14 (GPIO11)
- new net: JP7.2 (B), U13.16 (GPIO13)
- new net: TP8.1, U13.17 (GPIO14)
- new net: TP8.1, U13.18 (GPIO15)
- new net: R22.1, TP9.1, U13.26 (RUN)
- new net: JP7.2 (B), U13.27 (GPIO16)
- new net: JP7.2 (B), U13.28 (GPIO17)
- new net: U13.51 (QSPI_SD3), U7.7 (IO3/RESET#)
- new net: U13.52 (QSPI_SCLK), U7.6 (SCK)
- new net: U13.53 (QSPI_SD0), U7.5 (SI/IO0)
- new net: U13.54 (QSPI_SD2), U7.3 (WP#/IO2)
- new net: U13.55 (QSPI_SD1), U7.2 (SO/IO1)
- new net: R22.1, U13.56 (QSPI_SS), U7.1 (CS#)
- new net RX: J3.4 (Pin_4), U13.2 (GPIO0)
- new net USB_DET: JP7.1 (A), JP7.2 (B), R22.1, R22.2, R22.2
- new net USB_SEL: JP7.1 (A), JP7.1 (A), R22.1, R22.2, TP9.1, U4.2 (SEL)
- no-connect marks 23 -> 48
Other:
- moved on the sheet: R22, TP11

Commit message: - power routed, locked
Parts:
- removed JP7: SolderJumper_2_Open, symbol Jumper:SolderJumper_2_Open
- added C32: 1u, Capacitor_SMD:C_0805_2012Metric_Pad1.18x1.45mm_HandSolder, symbol Device:C
Connections:
- net +3.3v: now also C32.1; no longer C4.1, C4.1, C4.1, C4.1, C4.1, C4.1, R22.2, R22.2, U7.8 (VCC)
- net GND: now also C32.2
- net at C27.2, L2.2: now also J4.1 (Pin_1); no longer J4.2 (Pin_2)
- net +Pico 3.3v: now reaches C32.1, U12.5 (VOUT), U13.1 (IOVDD), U13.10 (IOVDD), U13.22 (IOVDD), U13.33 (IOVDD), U13.42 (IOVDD), U13.43 (ADC_AVDD), U13.44 (VREG_IN), U13.48 (USB_VDD), U13.49 (IOVDD)
- net +Pico 3.3v: now also C4.1, C4.1, C4.1, C4.1, C4.1, C4.1, R22.2, R22.2, U7.8 (VCC)
- net at JP7.2 (B): now also U13.31 (GPIO20); no longer U13.15 (GPIO12)
- net at U13.13 (GPIO10): no longer JP7.2 (B)
- net at U13.14 (GPIO11): no longer JP7.2 (B)
- net at U13.16 (GPIO13): no longer JP7.2 (B)
- net at U13.17 (GPIO14): no longer TP8.1
- net at U13.18 (GPIO15): no longer TP8.1
- net at U13.27 (GPIO16): no longer JP7.2 (B)
- net at U13.28 (GPIO17): no longer JP7.2 (B)
- net at U13.29 (GPIO18): now also JP7.2 (B)
- net at U13.30 (GPIO19): now also JP7.2 (B)
- net at U13.32 (GPIO21): now also JP7.2 (B)
- net at U13.34 (GPIO22): now also TP8.1
- net at U13.35 (GPIO23): now also TP8.1
- net at U13.36 (GPIO24): now also JP7.2 (B)
- net at U13.37 (GPIO25): now also JP7.2 (B)
- net at C27.2, L3.2: now also J4.2 (Pin_2); no longer J4.1 (Pin_1)
- net at C27.2, L4.2: now also J4.3 (Pin_3); no longer J4.4 (Pin_4)
- net at C27.2, L5.2: now also J4.4 (Pin_4); no longer J4.3 (Pin_3)
- no-connect marks 48 -> 41
Other:
- moved on the sheet: C32, C4, JP7, R22, TP11, TP8, U12
